File: Inverter_KiCAD/Inverter_KiCAD.kicad_sch (KiCad schematic)
At the start: 12 parts, among them J101 Conn_02x19_Odd_Even, J102 Conn_01x03, J103 Conn_02x19_Odd_Even, J104 Conn_01x04

Commit message: rooting done
Parts:
- J102: footprint (none) -> Custom:691311700003
- J104: footprint (none) -> Custom:691311700004
Connections:
- net Earth: now also J102.1 (Pin_1); no longer J102.3 (Pin_3)
- net GND: now also J102.3 (Pin_3); no longer J102.1 (Pin_1)
Changed lines of the file:
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@@
   (junction (at 162.56 181.61) (diameter 0) (color 0 0 0 0)
-  )
-  (junction (at 189.23 106.68) (diameter 0) (color 0 0 0 0)
   )
   (junction (at 140.97 186.69) (diameter 0) (color 0 0 0 0)
@@
     (stroke (width 0) (type default))
   )
-  (wire (pts (xy 82.55 35.56) (xy 86.36 35.56))
+  (wire (pts (xy 83.82 35.56) (xy 86.36 35.56))
     (stroke (width 0) (type default))
   )
@@
     (stroke (width 0) (type default))
   )
-  (wire (pts (xy 82.55 33.02) (xy 102.87 33.02))
+  (wire (pts (xy 83.82 33.02) (xy 102.87 33.02))
     (stroke (width 0) (type default))
   )
@@
     (stroke (width 0) (type default))
   )
+  (wire (pts (xy 189.23 106.68) (xy 205.74 106.68))
+    (stroke (width 0) (type default))
+  )
   (wire (pts (xy 87.63 125.73) (xy 97.79 125.73))
     (stroke (width 0) (type default))
@@
     (stroke (width 0) (type default))
   )
-  (wire (pts (xy 189.23 106.68) (xy 205.74 106.68))
-    (stroke (width 0) (type default))
-  )
   (wire (pts (xy 195.58 46.99) (xy 204.47 46.99))
     (stroke (width 0) (type default))
@@
     (stroke (width 0) (type default))
   )
-  (wire (pts (xy 187.96 106.68) (xy 189.23 106.68))
-    (stroke (width 0) (type default))
-  )
   (wire (pts (xy 162.56 186.69) (xy 162.56 191.77))
     (stroke (width 0) (type default))
@@
     (stroke (width 0) (type default))
   )
-  (wire (pts (xy 82.55 30.48) (xy 85.09 30.48))
+  (wire (pts (xy 83.82 30.48) (xy 85.09 30.48))
     (stroke (width 0) (type default))
   )
@@
     )
   )
-  (symbol (lib_id "Connector_Generic:Conn_01x03") (at 77.47 33.02 0) (mirror y) (unit 1)
-    (in_bom yes) (on_board yes) (dnp no) (fields_autoplaced)
-    (property "Reference" "J102" (at 77.47 25.4 0)
-      (effects (font (size 1.27 1.27)))
-    )
-    (property "Value" "Conn_01x03" (at 77.47 27.94 0)
-      (effects (font (size 1.27 1.27)))
-    )
-    (property "Footprint" "" (at 77.47 33.02 0)
-      (effects (font (size 1.27 1.27)) hide)
-    )
-    (property "Datasheet" "https://www.we-online.com/components/products/datasheet/691311700003.pdf" (at 77.47 33.02 0)
-      (effects (font (size 1.27 1.27)) hide)
-    )
-    (property "MFR" "691311700003" (at 77.47 33.02 0)
-      (effects (font (size 1.27 1.27)) hide)
-    )
-    (pin "1")
-    (pin "2")
-    (pin "3")
-    (instances
-      (project "Inverter_KiCAD"
-        (path "/5e6c1e3f-0815-454a-8acb-8e3e2d064875"
-          (reference "J102") (unit 1)
-        )
-      )
-    )
-  )
   (symbol (lib_id "Mechanical:MountingHole_Pad") (at 137.16 191.77 90) (unit 1)
     (in_bom yes) (on_board yes) (dnp no)
@@
     )
   )
+  (symbol (lib_id "Connector_Generic:Conn_01x03") (at 78.74 33.02 180) (unit 1)
+    (in_bom yes) (on_board yes) (dnp no)
+    (property "Reference" "J102" (at 78.74 25.2541 0)
+      (effects (font (size 1.27 1.27)))
+    )
+    (property "Value" "Conn_01x03" (at 78.74 27.7941 0)
+      (effects (font (size 1.27 1.27)))
+    )
+    (property "Footprint" "Custom:691311700003" (at 78.74 33.02 0)
+      (effects (font (size 1.27 1.27)) hide)
+    )
+    (property "Datasheet" "https://www.we-online.com/components/products/datasheet/691311700003.pdf" (at 78.74 33.02 0)
+      (effects (font (size 1.27 1.27)) hide)
+    )
+    (property "MFR" "691311700003" (at 78.74 33.02 0)
+      (effects (font (size 1.27 1.27)) hide)
+    )
+    (pin "1")
+    (pin "2")
+    (pin "3")
+    (instances
+      (project "Inverter_KiCAD"
+        (path "/5e6c1e3f-0815-454a-8acb-8e3e2d064875"
+          (reference "J102") (unit 1)
+        )
+      )
+    )
+  )
   (symbol (lib_id "power:Earth") (at 261.62 40.64 180) (unit 1)
     (in_bom yes) (on_board yes) (dnp no) (fields_autoplaced)
@@
       (effects (font (size 1.27 1.27)) (justify left))
     )
-    (property "Footprint" "" (at 273.05 44.45 0)
+    (property "Footprint" "Custom:691311700004" (at 273.05 44.45 0)
       (effects (font (size 1.27 1.27)) hide)
     )
@@
       (effects (font (size 1.27 1.27)) (justify right))
     )
+    (pin "ISO_PWM_Break" input (at 189.23 120.65 0)
+      (effects (font (size 1.27 1.27)) (justify right))
+    )
+    (pin "USART1_TX" input (at 157.48 135.89 180)
+      (effects (font (size 1.27 1.27)) (justify left))
+    )
+    (pin "USART1_RX" input (at 157.48 133.35 180)
+      (effects (font (size 1.27 1.27)) (justify left))
+    )
+    (pin "ISO_PWM_Fan" input (at 189.23 118.11 0)
+      (effects (font (size 1.27 1.27)) (justify right))
+    )
+    (pin "I2C_SDA" input (at 189.23 110.49 0)
+      (effects (font (size 1.27 1.27)) (justify right))
+    )
+    (pin "I2C_SCL" input (at 189.23 113.03 0)
+      (effects (font (size 1.27 1.27)) (justify right))
+    )
     (pin "Pwr_Enable" input (at 189.23 106.68 0)
       (effects (font (size 1.27 1.27)) (justify right))
     )
-    (pin "ISO_PWM_Break" input (at 189.23 120.65 0)
-      (effects (font (size 1.27 1.27)) (justify right))
-    )
-    (pin "USART1_TX" input (at 157.48 135.89 180)
-      (effects (font (size 1.27 1.27)) (justify left))
-    )
-    (pin "USART1_RX" input (at 157.48 133.35 180)
-      (effects (font (size 1.27 1.27)) (justify left))
-    )
-    (pin "ISO_PWM_Fan" input (at 189.23 118.11 0)
-      (effects (font (size 1.27 1.27)) (justify right))
-    )
-    (pin "I2C_SDA" input (at 189.23 110.49 0)
-      (effects (font (size 1.27 1.27)) (justify right))
-    )
-    (pin "I2C_SCL" input (at 189.23 113.03 0)
-      (effects (font (size 1.27 1.27)) (justify right))
-    )

Commit message: apply changes
Parts:
- removed J102: Conn_01x03, Custom:691311700003, symbol Connector_Generic:Conn_01x03
- removed J104: Conn_01x04, Custom:691311700004, symbol Connector_Generic:Conn_01x04
- added J2: Conn_01x03, Custom:691311700003, symbol Connector_Generic:Conn_01x03
- added J901: Conn_01x02, Custom:691311700002, symbol Connector_Generic:Conn_01x02
Connections:
- net GND: now also J901.2 (Pin_2)
- net U_output: now also J2.1 (Pin_1)
- net VSupply_BB: now also J901.1 (Pin_1)
- net V_output: now also J2.2 (Pin_2)
- net W_output: now also J2.3 (Pin_3)
Changed lines of the file:
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@@
   (no_connect (at 88.9 120.65))
   (no_connect (at 27.94 113.03))
-  (wire (pts (xy 261.62 41.91) (xy 261.62 40.64))
-    (stroke (width 0) (type default))
-  )
   (wire (pts (xy 110.49 105.41) (xy 124.46 105.41))
     (stroke (width 0) (type default))
@@
     (stroke (width 0) (type default))
   )
-  (wire (pts (xy 83.82 35.56) (xy 86.36 35.56))
-    (stroke (width 0) (type default))
-  )
   (wire (pts (xy 110.49 123.19) (xy 124.46 123.19))
     (stroke (width 0) (type default))
@@
   )
   (wire (pts (xy 88.9 100.33) (xy 97.79 100.33))
-    (stroke (width 0) (type default))
-  )
-  (wire (pts (xy 261.62 41.91) (xy 267.97 41.91))
     (stroke (width 0) (type default))
   )
@@
   (label "PC8" (at 124.46 97.79 180) (fields_autoplaced)
     (effects (font (size 1.27 1.27)) (justify right bottom))
+  )
+  (symbol (lib_id "Connector_Generic:Conn_01x03") (at 273.05 46.99 0) (unit 1)
+    (in_bom yes) (on_board yes) (dnp no)
+    (property "Reference" "J2" (at 273.05 54.7559 0)
+      (effects (font (size 1.27 1.27)))
+    )
+    (property "Value" "Conn_01x03" (at 273.05 52.2159 0)
+      (effects (font (size 1.27 1.27)))
+    )
+    (property "Footprint" "Custom:691311700003" (at 273.05 46.99 0)
+      (effects (font (size 1.27 1.27)) hide)
+    )
+    (property "Datasheet" "https://www.we-online.com/components/products/datasheet/691311700003.pdf" (at 273.05 46.99 0)
+      (effects (font (size 1.27 1.27)) hide)
+    )
+    (property "MFR" "691311700003" (at 273.05 46.99 0)
+      (effects (font (size 1.27 1.27)) hide)
+    )
+    (pin "1")
+    (pin "2")
+    (pin "3")
+    (instances
+      (project "Inverter_KiCAD"
+        (path "/5e6c1e3f-0815-454a-8acb-8e3e2d064875"
+          (reference "J2") (unit 1)
+        )
+      )
+    )
   )
   (symbol (lib_id "power:GND") (at 121.92 49.53 270) (unit 1)
@@
     )
   )
-  (symbol (lib_id "power:Earth") (at 86.36 35.56 0) (unit 1)
-    (in_bom yes) (on_board yes) (dnp no) (fields_autoplaced)
-    (property "Reference" "#PWR0103" (at 86.36 41.91 0)
-      (effects (font (size 1.27 1.27)) hide)
-    )
-    (property "Value" "Earth" (at 86.36 39.37 0)
-      (effects (font (size 1.27 1.27)) hide)
-    )
-    (property "Footprint" "" (at 86.36 35.56 0)
-      (effects (font (size 1.27 1.27)) hide)
-    )
-    (property "Datasheet" "~" (at 86.36 35.56 0)
-      (effects (font (size 1.27 1.27)) hide)
-    )
-    (pin "1")
-    (instances
-      (project "Inverter_KiCAD"
-        (path "/5e6c1e3f-0815-454a-8acb-8e3e2d064875"
-          (reference "#PWR0103") (unit 1)
-        )
-      )
-    )
-  )
-  (symbol (lib_id "Connector_Generic:Conn_01x03") (at 78.74 33.02 180) (unit 1)
-    (in_bom yes) (on_board yes) (dnp no)
-    (property "Reference" "J102" (at 78.74 25.2541 0)
-      (effects (font (size 1.27 1.27)))
-    )
-    (property "Value" "Conn_01x03" (at 78.74 27.7941 0)
-      (effects (font (size 1.27 1.27)))
-    )
-    (property "Footprint" "Custom:691311700003" (at 78.74 33.02 0)
-      (effects (font (size 1.27 1.27)) hide)
-    )
-    (property "Datasheet" "https://www.we-online.com/components/products/datasheet/691311700003.pdf" (at 78.74 33.02 0)
-      (effects (font (size 1.27 1.27)) hide)
-    )
-    (property "MFR" "691311700003" (at 78.74 33.02 0)
-      (effects (font (size 1.27 1.27)) hide)
-    )
-    (pin "1")
-    (pin "2")
-    (pin "3")
-    (instances
-      (project "Inverter_KiCAD"
-        (path "/5e6c1e3f-0815-454a-8acb-8e3e2d064875"
-          (reference "J102") (unit 1)
-        )
-      )
-    )
-  )
-  (symbol (lib_id "power:Earth") (at 261.62 40.64 180) (unit 1)
-    (in_bom yes) (on_board yes) (dnp no) (fields_autoplaced)
-    (property "Reference" "#PWR0110" (at 261.62 34.29 0)
-      (effects (font (size 1.27 1.27)) hide)
-    )
-    (property "Value" "Earth" (at 261.62 36.83 0)
-      (effects (font (size 1.27 1.27)) hide)
-    )
-    (property "Footprint" "" (at 261.62 40.64 0)
-      (effects (font (size 1.27 1.27)) hide)
-    )
-    (property "Datasheet" "~" (at 261.62 40.64 0)
-      (effects (font (size 1.27 1.27)) hide)
-    )
-    (pin "1")
-    (instances
-      (project "Inverter_KiCAD"
-        (path "/5e6c1e3f-0815-454a-8acb-8e3e2d064875"
-          (reference "#PWR0110") (unit 1)
-        )
-      )
-    )
-  )
   (symbol (lib_id "Mechanical:MountingHole_Pad") (at 137.16 176.53 90) (unit 1)
     (in_bom yes) (on_board yes) (dnp no)
@@
     )
   )
-  (symbol (lib_id "Connector_Generic:Conn_01x04") (at 273.05 44.45 0) (unit 1)
-    (in_bom yes) (on_board yes) (dnp no)
-    (property "Reference" "J104" (at 267.97 35.56 0)
-      (effects (font (size 1.27 1.27)) (justify left))
-    )
-    (property "Value" "Conn_01x04" (at 267.97 38.1 0)
-      (effects (font (size 1.27 1.27)) (justify left))
-    )
-    (property "Footprint" "Custom:691311700004" (at 273.05 44.45 0)
-      (effects (font (size 1.27 1.27)) hide)
-    )
-    (property "Datasheet" "https://www.we-online.com/components/products/datasheet/691311700004.pdf" (at 273.05 44.45 0)
-      (effects (font (size 1.27 1.27)) hide)
-    )
-    (property "MFR" "691311700004" (at 273.05 44.45 0)
-      (effects (font (size 1.27 1.27)) hide)
-    )
-    (pin "1")
-    (pin "2")
-    (pin "3")
-    (pin "4")
-    (instances
-      (project "Inverter_KiCAD"
-        (path "/5e6c1e3f-0815-454a-8acb-8e3e2d064875"
-          (reference "J104") (unit 1)
-        )
-      )
-    )
-  )
   (symbol (lib_id "power:GND") (at 163.83 176.53 90) (unit 1)
     (in_bom yes) (on_board yes) (dnp no) (fields_autoplaced)
@@
         )
       )
+    )
+  )
+  (symbol (lib_id "Connector_Generic:Conn_01x02") (at 78.74 33.02 180) (unit 1)
+    (in_bom yes) (on_board yes) (dnp no)
+    (property "Reference" "J901" (at 78.74 25.4 0)
+      (effects (font (size 1.27 1.27)))
+    )
+    (property "Value" "Conn_01x02" (at 78.74 27.94 0)
+      (effects (font (size 1.27 1.27)))
+    )
+    (property "Footprint" "Custom:691311700002" (at 78.74 33.02 0)
+      (effects (font (size 1.27 1.27)) hide)
+    )
+    (property "Datasheet" "https://www.we-online.com/components/products/datasheet/691311700002.pdf" (at 78.74 33.02 0)
+      (effects (font (size 1.27 1.27)) hide)
+    )
+    (property "MFR" "691311700002" (at 78.74 33.02 0)
+      (effects (font (size 1.27 1.27)) hide)
+    )
+    (property "Field5" "" (at 78.74 33.02 0)
+      (effects (font (size 1.27 1.27)) hide)
+    )
+    (pin "1")
+    (pin "2")
+    (instances
+      (project "Inverter_KiCAD"
+        (path "/5e6c1e3f-0815-454a-8acb-8e3e2d064875/63722f1b-78db-4d3b-ade4-7dd7cc6c956f"
+          (reference "J901") (unit 1)
+        )
+        (path "/5e6c1e3f-0815-454a-8acb-8e3e2d064875"
+          (reference "J1") (unit 1)
+        )
+      )

Commit message: Update KiCAD
Other:
- note added: "691311500102"
- note added: "691311500103"
Changed lines of the file:
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@@
+    (effects (font (size 1.27 1.27)) (justify left bottom))
+  )
+  (text "691311500103" (at 264.16 39.37 0)
     (effects (font (size 1.27 1.27)) (justify left bottom))
   )
@@
     (effects (font (size 1.27 1.27)) (justify left bottom))
   )
+  (text "691311500102" (at 81.28 22.86 0)
+    (effects (font (size 1.27 1.27)) (justify left bottom))
+  )

Commit message: Update KiCAD
Other:
- note added: "nouvelle ref : 691311500102"
- note added: "nouvelle ref : 691311500103"
- note removed: "691311500102"
- note removed: "691311500103"
Changed lines of the file:
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@@
     (effects (font (size 1.27 1.27)) (justify left bottom))
   )
-  (text "691311500103" (at 264.16 39.37 0)
-    (effects (font (size 1.27 1.27)) (justify left bottom))
+  (text "nouvelle ref : \n691311500103" (at 256.54 39.37 0)
+    (effects (font (size 3.4 3.4) (thickness 0.762) bold) (justify left bottom))
   )
   (text "PA8" (at 92.71 125.73 0)
@@
     (effects (font (size 1.27 1.27)) (justify left bottom))
   )
-  (text "691311500102" (at 81.28 22.86 0)
-    (effects (font (size 1.27 1.27)) (justify left bottom))
+  (text "nouvelle ref : \n691311500102" (at 73.66 24.13 0)
+    (effects (font (size 3.4 3.4) (thickness 0.68) bold) (justify left bottom))
   )
   (text "E5V" (at 52.07 102.87 0)

Commit message: change pbs
Parts:
- J2: footprint Custom:691311700003 -> Custom:691311500103; MFR 691311700003 -> 691311700103
- J901: footprint Custom:691311700002 -> Custom:691311500102; MFR 691311700002 -> 691311700102
Other:
- note removed: "nouvelle ref : 691311500102"
- note removed: "nouvelle ref : 691311500103"
Changed lines of the file:
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@@
     (effects (font (size 1.27 1.27)) (justify left bottom))
-  )
-  (text "nouvelle ref : \n691311500103" (at 256.54 39.37 0)
-    (effects (font (size 3.4 3.4) (thickness 0.762) bold) (justify left bottom))
   )
   (text "PA8" (at 92.71 125.73 0)
@@
   (text "PD2" (at 52.07 100.33 0)
     (effects (font (size 1.27 1.27)) (justify left bottom))
-  )
-  (text "nouvelle ref : \n691311500102" (at 73.66 24.13 0)
-    (effects (font (size 3.4 3.4) (thickness 0.68) bold) (justify left bottom))
   )
   (text "E5V" (at 52.07 102.87 0)
@@
       (effects (font (size 1.27 1.27)))
     )
-    (property "Footprint" "Custom:691311700003" (at 273.05 46.99 0)
-      (effects (font (size 1.27 1.27)) hide)
-    )
-    (property "Datasheet" "https://www.we-online.com/components/products/datasheet/691311700003.pdf" (at 273.05 46.99 0)
-      (effects (font (size 1.27 1.27)) hide)
-    )
-    (property "MFR" "691311700003" (at 273.05 46.99 0)
+    (property "Footprint" "Custom:691311500103" (at 273.05 46.99 0)
+      (effects (font (size 1.27 1.27)) hide)
+    )
+    (property "Datasheet" "https://www.we-online.com/components/products/datasheet/691311500103.pdf" (at 273.05 46.99 0)
+      (effects (font (size 1.27 1.27)) hide)
+    )
+    (property "MFR" "691311700103" (at 273.05 46.99 0)
       (effects (font (size 1.27 1.27)) hide)
     )
@@
       (effects (font (size 1.27 1.27)))
     )
-    (property "Footprint" "Custom:691311700002" (at 78.74 33.02 0)
-      (effects (font (size 1.27 1.27)) hide)
-    )
-    (property "Datasheet" "https://www.we-online.com/components/products/datasheet/691311700002.pdf" (at 78.74 33.02 0)
-      (effects (font (size 1.27 1.27)) hide)
-    )
-    (property "MFR" "691311700002" (at 78.74 33.02 0)
-      (effects (font (size 1.27 1.27)) hide)
-    )
+    (property "Footprint" "Custom:691311500102" (at 78.74 33.02 0)
+      (effects (font (size 1.27 1.27)) hide)
+    )
+    (property "Datasheet" "https://www.we-online.com/components/products/datasheet/691311500102.pdf" (at 78.74 33.02 0)
+      (effects (font (size 1.27 1.27)) hide)
+    )
+    (property "MFR" "691311700102" (at 78.74 33.02 0)
+      (effects (font (size 1.27 1.27)) hide)
+    )
