File: Inverter_KiCAD/Inverter_KiCAD.kicad_sch (KiCad schematic)
At the start: 12 parts, among them J101 Conn_02x19_Odd_Even, J103 Conn_02x19_Odd_Even, J2 Conn_01x03, J901 Conn_01x02

Commit message: update pcb
Parts:
- H101, H102, H103, H104, H105, H106, H107, H108: MFR (none) -> -
- J101, J103: Fournisseur (none) -> Farnell; MFR (none) -> SSW-119-01-T-D; Ref (none) -> 2667437
- J104: renamed from J2; Fournisseur (none) -> Wurth; MFR 691311700103 -> 691 311 700 103
- J901: Fournisseur (none) -> Wurth; MFR 691311700102 -> 691 311 700 102
Connections:
- net GND: no longer H105.1, H106.1
- net VSupply_AB: now also H105.1, H106.1
Other:
- added sheet V_Power_LED (V_Power_LED.kicad_sch)
- sheet FAN ports: added ISO_5V; removed ISO_15V
- sheet MCU_STM32G474 ports: added Pwr_Enable_U, Pwr_Enable_V, Pwr_Enable_W; removed Pwr_Enable
- moved on the sheet: H105, H106, H107, H108

Commit message: add G474RE base project
Parts:
- added H109, H110, H111, H112, H113, H114: MountingHole_Pad, MountingHole:MountingHole_3.2mm_M3_Pad_Via, symbol Mechanical:MountingHole_Pad
Connections:
- net GND: now also H109.1, H110.1, H111.1, H112.1, H113.1, H114.1
Other:
- note added: "Heatsink"
- note added: "NUCLEO for student programming NUCLEO-G431RBT6"
- note removed: "NUCLEO for student programming"

Commit message: update pcb
Parts:
- J103: renamed from J101; footprint Connector_PinHeader_2.54mm:PinHeader_2x19_P2.54mm_Vertical -> Connector_PinSocket_2.54mm:PinSocket_2x19_P2.54mm_Vertical
- J104: renamed from J103; footprint Connector_PinHeader_2.54mm:PinHeader_2x19_P2.54mm_Vertical -> Connector_PinSocket_2.54mm:PinSocket_2x19_P2.54mm_Vertical
- renumbered H107 to H105, H108 to H106, H105 to H107, H106 to H108, J104 to J102, J901 to J?
Connections:
- net +3V3: now also J103.15 (Pin_15); no longer J103.16 (Pin_16)
- net +5V: now also J103.17 (Pin_17); no longer J103.18 (Pin_18)
- net 5V_USB_CHGR: now also J104.7 (Pin_7); no longer J104.8 (Pin_8)
- net AVDD: now also J104.8 (Pin_8); no longer J104.7 (Pin_7)
- net Bus_Imes: now also J103.36 (Pin_36); no longer J103.35 (Pin_35)
- net Bus_V: now also J103.27 (Pin_27); no longer J103.28 (Pin_28)
- net ENC_A: now also J104.14 (Pin_14); no longer J104.13 (Pin_13)
- net ENC_B: now also J103.31 (Pin_31); no longer J103.32 (Pin_32)
- net ENC_Z: now also J104.1 (Pin_1); no longer J104.2 (Pin_2)
- net IOREF: now also J103.11 (Pin_11); no longer J103.12 (Pin_12)
- net ISO_5V: now also J103.5 (Pin_5); no longer J103.6 (Pin_6)
- net ISO_GND: now also J103.21 (Pin_21), J103.7 (Pin_7), J104.10 (Pin_10), J104.19 (Pin_19), J104.31 (Pin_31); no longer J103.22 (Pin_22), J103.8 (Pin_8), J104.20 (Pin_20), J104.32 (Pin_32), J104.9 (Pin_9)
- net NUCLEO_NRST: now also J103.3 (Pin_3); no longer J103.4 (Pin_4)
- net NUCLEO_RX: now also J103.1 (Pin_1); no longer J103.2 (Pin_2)
- net NUCLEO_TX: now also J103.2 (Pin_2); no longer J103.1 (Pin_1)
- net PA11: now also J104.13 (Pin_13); no longer J104.14 (Pin_14)
- net PA12: now also J104.11 (Pin_11); no longer J104.12 (Pin_12)
- net PA13: now also J103.14 (Pin_14); no longer J103.13 (Pin_13)
- net PA14: now also J103.16 (Pin_16); no longer J103.15 (Pin_15)
- net PA15: now also J103.18 (Pin_18); no longer J103.17 (Pin_17)
- net PA5: now also J104.12 (Pin_12); no longer J104.11 (Pin_11)
- net PA7: now also J104.16 (Pin_16); no longer J104.15 (Pin_15)
- net PB10: now also J104.26 (Pin_26); no longer J104.25 (Pin_25)
- net PB11: now also J104.17 (Pin_17); no longer J104.18 (Pin_18)
- net PB12: now also J104.15 (Pin_15); no longer J104.16 (Pin_16)
- net PB2: now also J104.21 (Pin_21); no longer J104.22 (Pin_22)
- net PB3: now also J104.32 (Pin_32); no longer J104.31 (Pin_31)
- net PB4: now also J104.28 (Pin_28); no longer J104.27 (Pin_27)
- net PB5: now also J104.30 (Pin_30); no longer J104.29 (Pin_29)
- net PB6: now also J104.18 (Pin_18); no longer J104.17 (Pin_17)
- net PB7: now also J103.22 (Pin_22); no longer J103.21 (Pin_21)
- net PB8: now also J104.4 (Pin_4); no longer J104.3 (Pin_3)
- net PB8-BOOT0: now also J103.8 (Pin_8); no longer J103.7 (Pin_7)
- net PB9: now also J104.6 (Pin_6); no longer J104.5 (Pin_5)
- net PC12: now also J103.4 (Pin_4); no longer J103.3 (Pin_3)
- net PC13: now also J103.24 (Pin_24); no longer J103.23 (Pin_23)
- net PC14: now also J103.26 (Pin_26); no longer J103.25 (Pin_25)
- net PC15: now also J103.28 (Pin_28); no longer J103.27 (Pin_27)
- net PC4: now also J104.33 (Pin_33); no longer J104.34 (Pin_34)
- net PC4/PA2: now also J104.36 (Pin_36); no longer J104.35 (Pin_35)
- net PC5: now also J104.5 (Pin_5); no longer J104.6 (Pin_6)
- net PC5/PA3: now also J104.38 (Pin_38); no longer J104.37 (Pin_37)
- net PC6: now also J104.3 (Pin_3); no longer J104.4 (Pin_4)
- net PC7: now also J104.20 (Pin_20); no longer J104.19 (Pin_19)
- net PC9: now also J104.2 (Pin_2); no longer J104.1 (Pin_1)
- net PF0: now also J103.30 (Pin_30); no longer J103.29 (Pin_29)
- net PF1: now also J103.32 (Pin_32); no longer J103.31 (Pin_31)
- net U_Imes: now also J103.29 (Pin_29); no longer J103.30 (Pin_30)
- net U_PWM_H: now also J104.24 (Pin_24); no longer J104.23 (Pin_23)
- net U_PWM_L: now also J104.29 (Pin_29); no longer J104.30 (Pin_30)
- net U_VPh: now also J103.37 (Pin_37); no longer J103.38 (Pin_38)
- net VBAT: now also J103.34 (Pin_34); no longer J103.33 (Pin_33)
- net VDD: now also J103.6 (Pin_6); no longer J103.5 (Pin_5)
- net VIN: now also J103.23 (Pin_23); no longer J103.24 (Pin_24)
- net V_Imes: now also J104.23 (Pin_23); no longer J104.24 (Pin_24)
- net V_PWM_H: now also J104.22 (Pin_22); no longer J104.21 (Pin_21)
- net V_PWM_L: now also J104.27 (Pin_27); no longer J104.28 (Pin_28)
- net V_VPh: now also J103.38 (Pin_38); no longer J103.37 (Pin_37)
- net W_Imes: now also J103.33 (Pin_33); no longer J103.34 (Pin_34)
- net W_PWM_H: now also J104.34 (Pin_34); no longer J104.33 (Pin_33)
- net W_PWM_L: now also J104.25 (Pin_25); no longer J104.26 (Pin_26)
- net W_VPh: now also J103.35 (Pin_35); no longer J103.36 (Pin_36)
Other:
- note added: "MCU Side"
- note added: "NUCLEO for student programming NUCLEO-G474RE"
- note removed: "Isolated Side"
- note removed: "NUCLEO for student programming NUCLEO-G431RBT6"
- moved on the sheet: H101, H102, H103, H104, H105, H106, H107, H108, H109, H110, H111, H112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
