File: Inverter_KiCAD/Inverter_KiCAD.kicad_pcb (KiCad board)
At the start: 2 copper layers, 184 x 186 mm, 172 parts, among them J101 Conn_02x19_Odd_Even, J102 Conn_01x03, J103 Conn_02x19_Odd_Even, J104 Conn_01x04, J1101 Conn_01x02, J1102 Conn_01x02, J501 PX0580-PC-12132, J801 USB_C_Receptacle_USB2.0, J802 Conn_01x05, J803 Conn_ST_STDC14, J804 Conn_01x04, J901 Conn_01x02, Q1101 SQ2310ES, Q201 HCPL-315J-500E, Q202 IRF540N, Q203 IRF540N, Q301 HCPL-315J-500E, Q302 IRF540N, Q303 IRF540N, Q401 HCPL-315J-500E, Q402 IRF540N, Q403 IRF540N, Q901 BUK9637-100E, SW801 SW_Push, SW802 SW_Push, SW803 SW_Push, SW804 SW_Push, SW805 SW_Push, U1201 TCN75A, U201 MPRB2415S-6W, U202 MPRB2415S-6W, U203 HCPL-7800-500E, U204 GO 10-SME/SP3, U301 MPRB2415S-6W, U302 MPRB2415S-6W, U303 HCPL-7800-500E, U304 GO 10-SME/SP3, U401 MPRB2415S-6W, U402 MPRB2415S-6W, U403 HCPL-7800-500E, U404 GO 10-SME/SP3, U501 MP-LD30-23B12R2, U502 173010542, U503 AZ1117-3.3, U601 GO 10-SME/SP3, U602 HCPL-7800-500E, U701 17791063215, U801 STM32G474RETx, U802 USBLC6-2SC6, U901 ACPL-077L, U902 TC1412, Y801 16M

Commit message: change pcb
Parts:
- removed C1001, C1002, C1003, C1004: 1.5m, Capacitor_THT:CP_Radial_D35.0mm_P10.00mm_SnapIn
- moved C1005 144.3 mm to (197.0, 29.0), turned to -90 degrees
- moved C1009 144.3 mm to (53.0, 29.0), turned to -90 degrees
- moved C1006 72.7 mm to (161.0, 29.0), turned to -90 degrees
- moved C1008 72.7 mm to (89.0, 29.0), turned to -90 degrees
- moved C1007 10.0 mm to (125.0, 29.0), turned to -90 degrees

Commit message: apply changes
Parts:
- removed J102: Conn_01x03, Custom:691311700003
- removed J104: Conn_01x04, Custom:691311700004
- added D1: VS-15TQ060S-M3, Package_TO_SOT_SMD:TO-263-2, F.Cu at (23.2, 65.1)
- added J1: Conn_01x02, Custom:691311700002, F.Cu at (38.0, 94.5)
- added J2: Conn_01x03, Custom:691311700003, F.Cu at (228.6, 96.6)

Commit message: change pbs
Parts:
- J1: footprint Custom:691311700002 -> Custom:691311500102
- J2: footprint Custom:691311700003 -> Custom:691311500103
- moved D1 11.1 mm to (22.9, 76.2)
Connections:
- J501 pad 2: Earth -> unconnected-(J501-Earth-Pad2)
Routing:
- added copper zone on F.Cu, net /V_output
- removed copper zone on F.Cu, net /VSupply_AB
Other:
- copper layers 2 -> 4
Changed lines of the file:
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@@
   (layers
     (0 "F.Cu" signal)
+    (1 "In1.Cu" signal)
+    (2 "In2.Cu" signal)
     (31 "B.Cu" signal)
     (32 "B.Adhes" user "B.Adhesive")
@@
       (layer "F.Mask" (type "Top Solder Mask") (thickness 0.01))
       (layer "F.Cu" (type "copper") (thickness 0.035))
-      (layer "dielectric 1" (type "core") (thickness 1.51) (material "FR4") (epsilon_r 4.5) (loss_tangent 0.02))
+      (layer "dielectric 1" (type "prepreg") (thickness 0.1) (material "FR4") (epsilon_r 4.5) (loss_tangent 0.02))
+      (layer "In1.Cu" (type "copper") (thickness 0.035))
+      (layer "dielectric 2" (type "core") (thickness 1.24) (material "FR4") (epsilon_r 4.5) (loss_tangent 0.02))
+      (layer "In2.Cu" (type "copper") (thickness 0.035))
+      (layer "dielectric 3" (type "prepreg") (thickness 0.1) (material "FR4") (epsilon_r 4.5) (loss_tangent 0.02))
       (layer "B.Cu" (type "copper") (thickness 0.035))
       (layer "B.Mask" (type "Bottom Solder Mask") (thickness 0.01))
@@
   (net 44 "/MCU_STM32G474/USR_LED_4")
   (net 45 "Net-(D803-K)")
-  (net 46 "Earth")
+  (net 46 "unconnected-(J501-Earth-Pad2)")
   (net 47 "Net-(D804-K)")
   (net 48 "Net-(J501-N)")
@@
     )
   )
-  (footprint "Custom:691311700003" (layer "F.Cu")
+  (footprint "Custom:691311500103" (layer "F.Cu")
     (at 228.6 96.6 -90)
-    (property "MFR" "691311700003")
+    (descr "<b>WR-TBL Serie 311 - 5.08 mm Close Vertical PCB Header <br></b>Max Height = 12mm , Pitch 5.08mm , 3pins")
+    (property "MFR" "691311700103")
     (property "Sheetfile" "Inverter_KiCAD.kicad_sch")
     (property "Sheetname" "")
@@
     (property "ki_keywords" "connector")
     (attr through_hole)
-    (fp_text reference "J2" (at 0 -6 -90 unlocked) (layer "F.SilkS")
-        (effects (font (size 1 1) (thickness 0.1)))
-    )
-    (fp_text value "Conn_01x03" (at 0 5.5 -90 unlocked) (layer "F.Fab")
+    (fp_text reference "J2" (at 0 -5.135 -90) (layer "F.SilkS")
         (effects (font (size 1 1) (thickness 0.15)))
     )
-    (fp_text user "${REFERENCE}" (at 0 7 -90 unlocked) (layer "F.Fab")
+    (fp_text value "Conn_01x03" (at 4.12 5.865 -90) (layer "F.Fab")
         (effects (font (size 1 1) (thickness 0.15)))
     )
-    (fp_line (start -7.5 -3.7) (end -6.5 -4.7)
-      (stroke (width 0.1) (type default)) (layer "F.SilkS"))
-    (fp_rect (start -7.5 3.8) (end 7.5 -4.7)
-      (stroke (width 0.1) (type default)) (fill none) (layer "F.SilkS"))
-    (fp_rect (start -7.9 -5.1) (end 7.9 4.2)
-      (stroke (width 0.1) (type default)) (fill none) (layer "F.CrtYd"))
-    (pad "1" thru_hole circle (at -5 0 270) (size 3.2 3.2) (drill 1.6) (layers "*.Cu" "*.Mask")
+    (fp_line (start -8.72 -3.9) (end 8.72 -3.9)
+      (stroke (width 0.2) (type solid)) (layer "F.SilkS"))
+    (fp_line (start -8.72 4.8) (end -8.72 -3.9)
+      (stroke (width 0.2) (type solid)) (layer "F.SilkS"))
+    (fp_line (start 8.72 -3.9) (end 8.72 4.8)
+      (stroke (width 0.2) (type solid)) (layer "F.SilkS"))
+    (fp_line (start 8.72 4.8) (end -8.72 4.8)
+      (stroke (width 0.2) (type solid)) (layer "F.SilkS"))
+    (fp_circle (center -6.84 -2) (end -6.74 -2)
+      (stroke (width 0.4) (type solid)) (fill none) (layer "F.SilkS"))
+    (fp_poly
+      (pts
+        (xy -8.92 -4.1)
+        (xy 8.92 -4.1)
+        (xy 8.92 5)
+        (xy -8.925 5)
+      )
+      (stroke (width 0.1) (type solid)) (fill none) (layer "F.CrtYd"))
+    (fp_line (start -8.62 -3.8) (end -8.62 4.7)
+      (stroke (width 0.1) (type solid)) (layer "F.Fab"))
+    (fp_line (start -8.62 4.7) (end 8.62 4.7)
+      (stroke (width 0.1) (type solid)) (layer "F.Fab"))
+    (fp_line (start 8.62 -3.8) (end -8.62 -3.8)
+      (stroke (width 0.1) (type solid)) (layer "F.Fab"))
+    (fp_line (start 8.62 4.7) (end 8.62 -3.8)
+      (stroke (width 0.1) (type solid)) (layer "F.Fab"))
+    (pad "1" thru_hole circle (at -5.08 0 270) (size 2.4 2.4) (drill 1.6) (layers "*.Cu" "*.Mask")
       (net 103 "/U_output") (pinfunction "Pin_1") (pintype "passive"))
-    (pad "2" thru_hole circle (at 0 0 270) (size 3.2 3.2) (drill 1.6) (layers "*.Cu" "*.Mask")
+    (pad "2" thru_hole circle (at 0 0 270) (size 2.4 2.4) (drill 1.6) (layers "*.Cu" "*.Mask")
       (net 104 "/V_output") (pinfunction "Pin_2") (pintype "passive"))
-    (pad "3" thru_hole circle (at 5 0 270) (size 3.2 3.2) (drill 1.6) (layers "*.Cu" "*.Mask")
+    (pad "3" thru_hole circle (at 5.08 0 270) (size 2.4 2.4) (drill 1.6) (layers "*.Cu" "*.Mask")
       (net 105 "/W_output") (pinfunction "Pin_3") (pintype "passive"))
   )
@@
       (net 48 "Net-(J501-N)") (pinfunction "N") (pintype "power_out"))
     (pad "2" thru_hole circle (at 0 4.825 90) (size 3.2 3.2) (drill 1.6) (layers "*.Cu" "*.Mask")
-      (net 46 "Earth") (pinfunction "Earth") (pintype "power_out"))
+      (net 46 "unconnected-(J501-Earth-Pad2)") (pinfunction "Earth") (pintype "power_out+no_connect"))
     (pad "3" thru_hole circle (at 9.14 4.825 90) (size 3.2 3.2) (drill 1.6) (layers "*.Cu" "*.Mask")
       (net 49 "Net-(J501-L)") (pinfunction "L") (pintype "power_out"))
@@
   )
   (footprint "Package_TO_SOT_SMD:TO-263-2" (layer "F.Cu")
-    (at 23.225 65.075 90)
+    (at 22.86 76.2 90)
     (descr "TO-263/D2PAK/DDPAK SMD package, http://www.infineon.com/cms/en/product/packages/PG-TO263/PG-TO263-3-1/")
     (tags "D2PAK DDPAK TO-263 D2PAK-3 TO-263-3 SOT-404")
@@
       (net 6 "GND") (pinfunction "1") (pintype "input"))
   )
-  (footprint "Custom:691311700002" (layer "F.Cu")
+  (footprint "Custom:691311500102" (layer "F.Cu")
     (at 38 94.5 90)
+    (descr "<b>WR-TBL Serie 311 - 5.08 mm Close Vertical PCB Header , 2 Pins")
     (property "Field5" "")
-    (property "MFR" "691311700002")
+    (property "MFR" "691311700102")
     (property "Sheetfile" "Inverter_KiCAD.kicad_sch")
     (property "Sheetname" "")
@@
     (property "ki_keywords" "connector")
     (attr through_hole)
-    (fp_text reference "J1" (at 0 -6 90 unlocked) (layer "F.SilkS")
-        (effects (font (size 1 1) (thickness 0.1)))
+    (fp_text reference "J1" (at 0.289 -5.4235 90) (layer "F.SilkS")
+        (effects (font (size 1 1) (thickness 0.15)))
     )
-    (fp_text value "Conn_01x02" (at 0 5.5 90 unlocked) (layer "F.Fab")
+    (fp_text value "Conn_01x02" (at 3.984 5.9316 90) (layer "F.Fab")
         (effects (font (size 1 1) (thickness 0.15)))
     )
-    (fp_text user "${REFERENCE}" (at 0 7 90 unlocked) (layer "F.Fab")
+    (fp_text user "1" (at -3 3 90) (layer "Dwgs.User")
         (effects (font (size 1 1) (thickness 0.15)))
     )
-    (fp_line (start -5 -3.7) (end -4 -4.7)
-      (stroke (width 0.1) (type default)) (layer "F.SilkS"))
-    (fp_rect (start -5 3.8) (end 5 -4.7)
-      (stroke (width 0.1) (type default)) (fill none) (layer "F.SilkS"))
-    (fp_rect (start -5.4 -5.1) (end 5.4 4.2)
-      (stroke (width 0.1) (type default)) (fill none) (layer "F.CrtYd"))
-    (pad "1" thru_hole circle (at -2.5 0 90) (size 3.2 3.2) (drill 1.6) (layers "*.Cu" "*.Mask")
+    (fp_line (start -6.08 -3.8) (end -6.08 4.7)
+      (stroke (width 0.127) (type solid)) (layer "F.SilkS"))
+    (fp_line (start -6.08 4.7) (end 6.08 4.7)
+      (stroke (width 0.127) (type solid)) (layer "F.SilkS"))
+    (fp_line (start 6.08 -3.8) (end -6.08 -3.8)
+      (stroke (width 0.127) (type solid)) (layer "F.SilkS"))
+    (fp_line (start 6.08 4.7) (end 6.08 -3.8)
+      (stroke (width 0.127) (type solid)) (layer "F.SilkS"))
+    (fp_poly
+      (pts
+        (xy -6.33 -4.05)
+        (xy 6.33 -4.05)
+        (xy 6.33 4.95)
+        (xy -6.33 4.95)
+      )
+      (stroke (width 0.127) (type solid)) (fill none) (layer "F.CrtYd"))
+    (pad "1" thru_hole circle (at -2.54 0 90) (size 2.4 2.4) (drill 1.6) (layers "*.Cu" "*.Mask")
       (net 7 "/VSupply_BB") (pinfunction "Pin_1") (pintype "passive"))
-    (pad "2" thru_hole circle (at 2.5 0 90) (size 3.2 3.2) (drill 1.6) (layers "*.Cu" "*.Mask")
+    (pad "2" thru_hole circle (at 2.54 0 90) (size 2.4 2.4) (drill 1.6) (layers "*.Cu" "*.Mask")
       (net 6 "GND") (pinfunction "Pin_2") (pintype "passive"))
   )
@@
     )
   )
-  (zone (net 36) (net_name "/VSupply_AB") (layer "F.Cu") (hatch edge 0.5)
+  (zone (net 104) (net_name "/V_output") (layer "F.Cu") (hatch edge 0.5)
     (priority 4)
-    (connect_pads yes (clearance 0.5))
+    (connect_pads yes (clearance 1))
     (min_thickness 0.25) (filled_areas_thickness no)
     (fill yes (thermal_gap 0.5) (thermal_bridge_width 0.5))
@@
   (zone (net 6) (net_name "GND") (layers "F&B.Cu") (hatch edge 0.5)
     (priority 1)
-    (connect_pads (clearance 0.5))
+    (connect_pads yes (clearance 1))
     (min_thickness 0.25) (filled_areas_thickness no)
     (fill yes (thermal_gap 0.5) (thermal_bridge_width 0.5))
@@
   (zone (net 76) (net_name "/Vbus") (layer "B.Cu") (hatch edge 0.5)
     (priority 3)
-    (connect_pads yes (clearance 0.5))
+    (connect_pads yes (clearance 1))
     (min_thickness 0.25) (filled_areas_thickness no)
     (fill yes (thermal_gap 0.5) (thermal_bridge_width 0.5))

Commit message: v0 PCB
Parts:
- removed J1: Conn_01x02, Custom:691311500102
- added C1301: 100n, Capacitor_SMD:C_0402_1005Metric_Pad0.74x0.62mm_HandSolder, B.Cu at (192.6, 151.3)
- added C206: 10u, Capacitor_SMD:C_0805_2012Metric, F.Cu at (83.5, 103.9)
- added C306: 10u, Capacitor_SMD:C_0805_2012Metric, F.Cu at (131.1, 103.8)
- added C406: 10u, Capacitor_SMD:C_0805_2012Metric, F.Cu at (178.6, 103.8)
- added J102: Conn_01x02, Custom:691311500102, F.Cu at (42.5, 74.3)
- added J1301: DE9_Receptacle_MountingHoles, Custom:618009233821, F.Cu at (204.2, 149.5)
- added J1302: Conn_01x03, Connector_PinHeader_2.54mm:PinHeader_1x03_P2.54mm_Vertical, F.Cu at (194.4, 148.1)
- added U1301: MAX3097ECSE+, Package_SO:SOIC-16_3.9x9.9mm_P1.27mm, B.Cu at (196.9, 155.2)
- J901: footprint Custom:691311700002 -> Custom:691311500102
- moved D903 35.9 mm to (57.7, 84.8), turned to 0 degrees
- moved D902 21.7 mm to (57.7, 73.3)
- moved R903 18.1 mm to (44.9, 94.7), turned to 0 degrees
- moved J104 17.2 mm to (212.0, 92.0)
- moved H108 17.2 mm to (47.0, 58.0)
- moved Q901 15.6 mm to (57.7, 96.3), turned to 0 degrees
- moved J901 5.77 mm to (42.5, 87.1)
- moved C813 0.22 mm to (127.7, 138.6)
- renumbered C1005 to C1001, C1006 to C1002, C1007 to C1003, C1008 to C1004, C1009 to C1005, C206 to C207, C207 to C208, C208 to C209, C209 to C210, C210 to C211, C306 to C307, C307 to C308, C308 to C309, C309 to C310, C310 to C311, C406 to C407, C407 to C408, C408 to C409, C409 to C410, C410 to C411, D1 to D903, J2 to J104
Connections:
- net /MCU_STM32G474/ENC_A renamed /MCU_STM32G474/ENC_BTN_A
- net /MCU_STM32G474/ENC_B renamed /MCU_STM32G474/ENC_BTN_B
- net /MCU_STM32G474/ENC_BTN renamed /MCU_STM32G474/ENC_BTN_P
- H101 pad 1: /ISO_GND -> unconnected-(H101-Pad1)
- J101 pad 32: /PA4 -> /ENC_B
- J103 pad 13: /PA6 -> /ENC_A
- J103 pad 2: /PC8 -> /ENC_Z
- U801 pad 10: unconnected-(U801-PC2-Pad10) -> /ENC_Z
- U801 pad 11: unconnected-(U801-PC3-Pad11) -> /V_VPh
- U801 pad 26: unconnected-(U801-PB2-Pad26) -> /V_Imes
- U801 pad 8: /V_VPh -> /ENC_A
- U801 pad 9: /V_Imes -> /ENC_B
Routing:
- net /ISO_3V3: track 378.1 -> 237.1 mm, vias 17 -> 19
- net /ENC_Z: track 0.00 -> 104.2 mm, vias 0 -> 3
- net /ENC_B: track 0.00 -> 98.8 mm, vias 0 -> 3
- net /ISO_GND: track 93.7 -> 184.1 mm, vias 45 -> 61
- net /ENC_A: track 0.00 -> 89.6 mm, vias 0 -> 3
- net /Vbus: track 78.2 -> 19.0 mm, vias 59 -> 33
- net /VSupply_AB: track 0.00 -> 30.6 mm, vias 42 -> 0
- net /ISO_5V: track 216.7 -> 242.2 mm
- net /encoderMotor/VCC_Enc: track 0.00 -> 20.8 mm
- net /break/PWM_Mosfet: track 33.7 -> 21.5 mm
- net /Bus_V: track 160.3 -> 149.0 mm, vias 6 -> 5
- net /MCU_STM32G474/NRST: track 84.8 -> 74.7 mm
- net /MCU_STM32G474/SWO: track 78.6 -> 68.4 mm
- net /encoderMotor/B: track 0.00 -> 9.15 mm
- net /encoderMotor//Z: track 0.00 -> 8.20 mm
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- added copper zone on In2.Cu, net /ISO_3V3
- added copper zone on In1.Cu, net /ISO_GND
- added copper zone on F.Cu, net /VSupply_AB
- added copper zone on In1.Cu, net /Vbus
- added copper zone on In2.Cu, net /Vbus
- added copper zone on In1.Cu, net GND
- added copper zone on In2.Cu, net GND
- removed copper zone on B.Cu, net /VSupply_AB
- removed copper zone on F.Cu, net /V_output
Other:
- board text added: "1"
