File: Inverter_KiCAD/_autosave-Inverter_KiCAD.kicad_sch (KiCad schematic)
At the start: 12 parts, among them J101 Conn_02x19_Odd_Even, J103 Conn_02x19_Odd_Even, J2 Conn_01x03, J901 Conn_01x02

Commit message: v0 PCB
Parts:
- renumbered J2 to J104
Changed lines of the file:
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@@
   (symbol (lib_id "Connector_Generic:Conn_01x03") (at 386.08 90.17 0) (unit 1)
     (in_bom yes) (on_board yes) (dnp no)
-    (property "Reference" "J2" (at 386.08 97.9359 0)
+    (property "Reference" "J104" (at 386.08 97.9359 0)
       (effects (font (size 1.27 1.27)))
     )
@@
       (project "Inverter_KiCAD"
         (path "/5e6c1e3f-0815-454a-8acb-8e3e2d064875"
-          (reference "J2") (unit 1)
+          (reference "J104") (unit 1)
         )
       )
@@
   (symbol (lib_id "power:GND") (at 170.18 46.99 0) (unit 1)
     (in_bom yes) (on_board yes) (dnp no) (fields_autoplaced)
-    (property "Reference" "#PWR0111" (at 170.18 53.34 0)
+    (property "Reference" "#PWR0104" (at 170.18 53.34 0)
       (effects (font (size 1.27 1.27)) hide)
     )
@@
       (project "Inverter_KiCAD"
         (path "/5e6c1e3f-0815-454a-8acb-8e3e2d064875"
-          (reference "#PWR0111") (unit 1)
+          (reference "#PWR0104") (unit 1)
         )
       )
@@
   (symbol (lib_id "power:GND") (at 243.84 43.18 0) (unit 1)
     (in_bom yes) (on_board yes) (dnp no) (fields_autoplaced)
-    (property "Reference" "#PWR0109" (at 243.84 49.53 0)
+    (property "Reference" "#PWR0106" (at 243.84 49.53 0)
       (effects (font (size 1.27 1.27)) hide)
     )
@@
       (project "Inverter_KiCAD"
         (path "/5e6c1e3f-0815-454a-8acb-8e3e2d064875"
-          (reference "#PWR0109") (unit 1)
+          (reference "#PWR0106") (unit 1)
         )
       )
@@
   (symbol (lib_id "power:GND") (at 95.25 60.96 90) (unit 1)
     (in_bom yes) (on_board yes) (dnp no) (fields_autoplaced)
-    (property "Reference" "#PWR0104" (at 101.6 60.96 0)
+    (property "Reference" "#PWR0103" (at 101.6 60.96 0)
       (effects (font (size 1.27 1.27)) hide)
     )
@@
       (project "Inverter_KiCAD"
         (path "/5e6c1e3f-0815-454a-8acb-8e3e2d064875"
-          (reference "#PWR0104") (unit 1)
+          (reference "#PWR0103") (unit 1)
         )
       )
@@
   (symbol (lib_id "power:GND") (at 375.92 130.81 90) (unit 1)
     (in_bom yes) (on_board yes) (dnp no) (fields_autoplaced)
-    (property "Reference" "#PWR0106" (at 382.27 130.81 0)
+    (property "Reference" "#PWR0109" (at 382.27 130.81 0)
       (effects (font (size 1.27 1.27)) hide)
     )
@@
       (project "Inverter_KiCAD"
         (path "/5e6c1e3f-0815-454a-8acb-8e3e2d064875"
-          (reference "#PWR0106") (unit 1)
+          (reference "#PWR0109") (unit 1)
         )
       )
@@
         )
         (path "/5e6c1e3f-0815-454a-8acb-8e3e2d064875"
-          (reference "J1") (unit 1)
-        )
-      )
+          (reference "J102") (unit 1)
+        )
+      )
