File: Inverter_KiCAD/FAN.kicad_sch (KiCad schematic)
At the start: 5 parts

Commit message: update pcb
Parts:
- J? (x2): Fournisseur (none) -> Stock
- Q?: Fournisseur (none) -> RS; MFR (none) -> SQ2310ES-T1_BE3; Ref (none) -> 787-9443
- R?: footprint Resistor_SMD:R_0402_1005Metric_Pad0.72x0.64mm_HandSolder -> Resistor_SMD:R_0402_1005Metric; symbol Device:R_Small_US -> Device:R_Small; Fournisseur (none) -> Stock
- R?: footprint Resistor_SMD:R_0402_1005Metric_Pad0.72x0.64mm_HandSolder -> Resistor_SMD:R_0402_1005Metric; Fournisseur (none) -> Farnell; MFR (none) -> MC00625W0402110K; Ref (none) -> 2130433
Connections:
- net ISO_15V renamed ISO_5V
Changed lines of the file:
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@@
     (stroke (width 0) (type default))
   )
-  (hierarchical_label "ISO_15V" (shape input) (at 53.34 25.4 90) (fields_autoplaced)
+  (hierarchical_label "ISO_5V" (shape input) (at 53.34 25.4 90) (fields_autoplaced)
     (effects (font (size 1.27 1.27)) (justify left))
   )
@@
     )
     (property "Datasheet" "~" (at 50.8 38.1 0)
+      (effects (font (size 1.27 1.27)) hide)
+    )
+    (property "Fournisseur" "RS" (at 50.8 38.1 0)
+      (effects (font (size 1.27 1.27)) hide)
+    )
+    (property "MFR" "SQ2310ES-T1_BE3" (at 50.8 38.1 0)
+      (effects (font (size 1.27 1.27)) hide)
+    )
+    (property "Ref" "787-9443" (at 50.8 38.1 0)
       (effects (font (size 1.27 1.27)) hide)
     )
@@
     )
   )
-  (symbol (lib_id "Device:R_Small_US") (at 40.64 38.1 270) (unit 1)
+  (symbol (lib_id "Device:R_Small") (at 40.64 38.1 270) (unit 1)
     (in_bom yes) (on_board yes) (dnp no)
     (property "Reference" "R?" (at 36.83 36.83 90)
@@
       (effects (font (size 1.27 1.27)) (justify right))
     )
-    (property "Footprint" "Resistor_SMD:R_0402_1005Metric_Pad0.72x0.64mm_HandSolder" (at 40.64 38.1 0)
+    (property "Footprint" "Resistor_SMD:R_0402_1005Metric" (at 40.64 38.1 0)
       (effects (font (size 1.27 1.27)) hide)
     )
     (property "Datasheet" "~" (at 40.64 38.1 0)
+      (effects (font (size 1.27 1.27)) hide)
+    )
+    (property "Fournisseur" "Stock" (at 40.64 38.1 0)
       (effects (font (size 1.27 1.27)) hide)
     )
@@
       (effects (font (size 1.27 1.27)) hide)
     )
+    (property "Fournisseur" "Stock" (at 46.99 29.21 0)
+      (effects (font (size 1.27 1.27)) hide)
+    )
     (pin "1")
     (pin "2")
@@
       (effects (font (size 1.27 1.27)) hide)
     )
+    (property "Fournisseur" "Stock" (at 59.69 29.21 0)
+      (effects (font (size 1.27 1.27)) hide)
+    )
     (pin "1")
     (pin "2")
@@
       (effects (font (size 1.27 1.27)) (justify right))
     )
-    (property "Footprint" "Resistor_SMD:R_0402_1005Metric_Pad0.72x0.64mm_HandSolder" (at 44.45 41.91 0)
+    (property "Footprint" "Resistor_SMD:R_0402_1005Metric" (at 44.45 41.91 0)
       (effects (font (size 1.27 1.27)) hide)
     )
@@
       (effects (font (size 1.27 1.27)) hide)
     )
+    (property "Fournisseur" "Farnell" (at 44.45 41.91 0)
+      (effects (font (size 1.27 1.27)) hide)
+    )
+    (property "MFR" "MC00625W0402110K" (at 44.45 41.91 0)
+      (effects (font (size 1.27 1.27)) hide)
+    )
+    (property "Ref" "2130433" (at 44.45 41.91 0)
+      (effects (font (size 1.27 1.27)) hide)
+    )
