File: Inverter_KiCAD/MCU_STM32G474.kicad_sch (KiCad schematic)
At the start: 42 parts, among them J801 USB_C_Receptacle_USB2.0, J802 Conn_01x05, J803 Conn_ST_STDC14, J804 Conn_01x04, SW801 SW_Push, SW802 SW_Push, SW803 SW_Push, SW804 SW_Push, SW805 SW_Push, U801 STM32G474RETx, U802 USBLC6-2SC6, Y801 16M

Commit message: end of sch, start pcb
Parts:
- C805: footprint Capacitor_SMD:C_0603_1608Metric_Pad1.08x0.95mm_HandSolder -> Capacitor_SMD:C_0402_1005Metric_Pad0.74x0.62mm_HandSolder
- R801, R802, R803, R804, R805, R806, R807: footprint Resistor_SMD:R_0603_1608Metric_Pad0.98x0.95mm_HandSolder -> Resistor_SMD:R_0402_1005Metric_Pad0.72x0.64mm_HandSolder
- Y801: footprint (none) -> Custom:ABLS-7.3728MHZ-CL-RESR-A-1-G-F
Connections:
- net USR_BTN_2: now also U801.18 (PA4); no longer U801.57 (PB4)
- net Screen_SCL renamed I2C_SCL
- net Screen_SDA renamed I2C_SDA
- new net ISO_PWM_Fan: U801.57 (PB4)
- no-connect marks 14 -> 13
Other:
- company: (none) -> ENSEA
- title: (none) -> AAP Inverter
Changed lines of the file:
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@@
 (kicad_sch (version 20230121) (generator eeschema)
   (paper "A4")
+  (title_block
+    (title "AAP Inverter")
+    (date "2023-05-01")
+    (company "ENSEA")
+  )
   (junction (at 175.26 46.99) (diameter 0) (color 0 0 0 0)
   )
@@
   (no_connect (at 234.95 41.91))
   (no_connect (at 62.23 104.14))
-  (no_connect (at 97.79 55.88))
   (wire (pts (xy 208.28 140.97) (xy 213.36 140.97))
     (stroke (width 0) (type default))
@@
     (stroke (width 0) (type default))
   )
+  (wire (pts (xy 97.79 55.88) (xy 110.49 55.88))
+    (stroke (width 0) (type default))
+  )
   (wire (pts (xy 250.19 128.27) (xy 261.62 128.27))
     (stroke (width 0) (type default))
@@
     (stroke (width 0) (type default))
   )
-  (wire (pts (xy 110.49 66.04) (xy 97.79 66.04))
+  (wire (pts (xy 97.79 66.04) (xy 113.03 66.04))
     (stroke (width 0) (type default))
   )
@@
     (stroke (width 0) (type default))
   )
-  (wire (pts (xy 110.49 68.58) (xy 97.79 68.58))
+  (wire (pts (xy 97.79 68.58) (xy 113.03 68.58))
     (stroke (width 0) (type default))
   )
@@
     (effects (font (size 1.27 1.27)) (justify right bottom))
   )
+  (label "I2C2_SCL" (at 213.36 151.13 0) (fields_autoplaced)
+    (effects (font (size 1.27 1.27)) (justify left bottom))
+  )
   (label "ISO_3V3A" (at 50.8 45.72 0) (fields_autoplaced)
     (effects (font (size 1.27 1.27)) (justify left bottom))
@@
     (effects (font (size 1.27 1.27)) (justify right bottom))
   )
-  (label "Screen_SCL" (at 213.36 151.13 0) (fields_autoplaced)
-    (effects (font (size 1.27 1.27)) (justify left bottom))
+  (label "USR_BTN_2" (at 110.49 55.88 180) (fields_autoplaced)
+    (effects (font (size 1.27 1.27)) (justify right bottom))
   )
   (label "VCP_TX" (at 110.49 114.3 180) (fields_autoplaced)
@@
     (effects (font (size 1.27 1.27)) (justify right bottom))
   )
-  (label "USR_BTN_2" (at 110.49 99.06 180) (fields_autoplaced)
-    (effects (font (size 1.27 1.27)) (justify right bottom))
-  )
   (label "D+" (at 213.36 92.71 180) (fields_autoplaced)
     (effects (font (size 1.27 1.27)) (justify right bottom))
@@
     (effects (font (size 1.27 1.27)) (justify right bottom))
   )
-  (label "Screen_SDA" (at 213.36 153.67 0) (fields_autoplaced)
-    (effects (font (size 1.27 1.27)) (justify left bottom))
-  )
   (label "USR_BTN_1" (at 50.8 63.5 0) (fields_autoplaced)
     (effects (font (size 1.27 1.27)) (justify left bottom))
@@
     (effects (font (size 1.27 1.27)) (justify right bottom))
   )
-  (label "Screen_SCL" (at 110.49 68.58 180) (fields_autoplaced)
+  (label "I2C2_SDA" (at 213.36 153.67 0) (fields_autoplaced)
+    (effects (font (size 1.27 1.27)) (justify left bottom))
+  )
+  (label "I2C2_SCL" (at 110.49 68.58 180) (fields_autoplaced)
     (effects (font (size 1.27 1.27)) (justify right bottom))
   )
@@
     (effects (font (size 1.27 1.27)) (justify right bottom))
   )
-  (label "Screen_SDA" (at 110.49 66.04 180) (fields_autoplaced)
+  (label "I2C2_SDA" (at 110.49 66.04 180) (fields_autoplaced)
     (effects (font (size 1.27 1.27)) (justify right bottom))
   )
@@
     (effects (font (size 1.27 1.27)) (justify left))
   )
+  (hierarchical_label "ISO_PWM_Fan" (shape input) (at 110.49 99.06 0) (fields_autoplaced)
+    (effects (font (size 1.27 1.27)) (justify left))
+  )
+  (hierarchical_label "I2C_SCL" (shape input) (at 113.03 68.58 0) (fields_autoplaced)
+    (effects (font (size 1.27 1.27)) (justify left))
+  )
   (hierarchical_label "IC_PWN_U_H" (shape input) (at 97.79 50.8 0) (fields_autoplaced)
     (effects (font (size 1.27 1.27)) (justify left))
@@
     (effects (font (size 1.27 1.27)) (justify left))
   )
+  (hierarchical_label "I2C_SDA" (shape input) (at 113.03 66.04 0) (fields_autoplaced)
+    (effects (font (size 1.27 1.27)) (justify left))
+  )
   (symbol (lib_id "Device:R_Small") (at 273.05 33.02 90) (unit 1)
     (in_bom yes) (on_board yes) (dnp no) (fields_autoplaced)
@@
       (effects (font (size 1.27 1.27)))
     )
-    (property "Footprint" "Resistor_SMD:R_0603_1608Metric_Pad0.98x0.95mm_HandSolder" (at 273.05 33.02 0)
+    (property "Footprint" "Resistor_SMD:R_0402_1005Metric_Pad0.72x0.64mm_HandSolder" (at 273.05 33.02 0)
       (effects (font (size 1.27 1.27)) hide)
     )
@@
       (effects (font (size 1.27 1.27)) (justify left))
     )
-    (property "Footprint" "Resistor_SMD:R_0603_1608Metric_Pad0.98x0.95mm_HandSolder" (at 189.23 91.44 0)
+    (property "Footprint" "Resistor_SMD:R_0402_1005Metric_Pad0.72x0.64mm_HandSolder" (at 189.23 91.44 0)
       (effects (font (size 1.27 1.27)) hide)
     )
@@
       (effects (font (size 1.27 1.27)) (justify right))
     )
-    (property "Footprint" "" (at 38.1 57.15 0)
+    (property "Footprint" "Custom:ABLS-7.3728MHZ-CL-RESR-A-1-G-F" (at 38.1 57.15 0)
       (effects (font (size 1.27 1.27)) hide)
     )
@@
       (effects (font (size 1.27 1.27)))
     )
-    (property "Footprint" "Resistor_SMD:R_0603_1608Metric_Pad0.98x0.95mm_HandSolder" (at 113.03 109.22 0)
+    (property "Footprint" "Resistor_SMD:R_0402_1005Metric_Pad0.72x0.64mm_HandSolder" (at 113.03 109.22 0)
       (effects (font (size 1.27 1.27)) hide)
     )
@@
       (effects (font (size 1.27 1.27)))
     )
-    (property "Footprint" "Resistor_SMD:R_0603_1608Metric_Pad0.98x0.95mm_HandSolder" (at 273.05 41.91 0)
+    (property "Footprint" "Resistor_SMD:R_0402_1005Metric_Pad0.72x0.64mm_HandSolder" (at 273.05 41.91 0)
       (effects (font (size 1.27 1.27)) hide)
     )
@@
       (effects (font (size 1.27 1.27)) (justify left))
     )
-    (property "Footprint" "Resistor_SMD:R_0603_1608Metric_Pad0.98x0.95mm_HandSolder" (at 189.23 83.82 0)
+    (property "Footprint" "Resistor_SMD:R_0402_1005Metric_Pad0.72x0.64mm_HandSolder" (at 189.23 83.82 0)
       (effects (font (size 1.27 1.27)) hide)
     )
@@
       (effects (font (size 1.27 1.27)))
     )
-    (property "Footprint" "Resistor_SMD:R_0603_1608Metric_Pad0.98x0.95mm_HandSolder" (at 273.05 50.8 0)
+    (property "Footprint" "Resistor_SMD:R_0402_1005Metric_Pad0.72x0.64mm_HandSolder" (at 273.05 50.8 0)
       (effects (font (size 1.27 1.27)) hide)
     )
@@
       (effects (font (size 1.27 1.27)) (justify left))
     )
-    (property "Footprint" "Capacitor_SMD:C_0603_1608Metric_Pad1.08x0.95mm_HandSolder" (at 166.37 50.8 0)
+    (property "Footprint" "Capacitor_SMD:C_0402_1005Metric_Pad0.74x0.62mm_HandSolder" (at 166.37 50.8 0)
       (effects (font (size 1.27 1.27)) hide)
     )
@@
       (effects (font (size 1.27 1.27)))
     )
-    (property "Footprint" "Resistor_SMD:R_0603_1608Metric_Pad0.98x0.95mm_HandSolder" (at 273.05 24.13 0)
-      (effects (font (size 1.27 1.27)) hide)
-    )
+    (property "Footprint" "Resistor_SMD:R_0402_1005Metric_Pad0.72x0.64mm_HandSolder" (at 273.05 24.13 0)
+      (effects (font (size 1.27 1.27)) hide)
+    )

Commit message: rooting done
Parts:
- SW801, SW802, SW803, SW804, SW805: footprint Button_Switch_SMD:SW_SPST_B3U-3000P -> Custom:435451019820
Connections:
- net ISO_GND: now also J801.S1 (SHIELD)
- no-connect marks 13 -> 12
Changed lines of the file:
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@@
     (company "ENSEA")
+  )
+  (junction (at 161.29 119.38) (diameter 0) (color 0 0 0 0)
   )
   (junction (at 175.26 46.99) (diameter 0) (color 0 0 0 0)
@@
   (no_connect (at 62.23 73.66))
   (no_connect (at 97.79 71.12))
-  (no_connect (at 153.67 119.38))
   (no_connect (at 176.53 111.76))
   (no_connect (at 62.23 76.2))
@@
     (stroke (width 0) (type default))
   )
+  (wire (pts (xy 153.67 119.38) (xy 161.29 119.38))
+    (stroke (width 0) (type default))
+  )
   (wire (pts (xy 184.15 86.36) (xy 184.15 83.82))
     (stroke (width 0) (type default))
@@
       (effects (font (size 1.27 1.27)))
     )
-    (property "Footprint" "Button_Switch_SMD:SW_SPST_B3U-3000P" (at 264.16 97.79 0)
+    (property "Footprint" "Custom:435451019820" (at 264.16 97.79 0)
       (effects (font (size 1.27 1.27)) hide)
     )
@@
       (effects (font (size 1.27 1.27)))
     )
-    (property "Footprint" "Button_Switch_SMD:SW_SPST_B3U-3000P" (at 264.16 80.01 0)
+    (property "Footprint" "Custom:435451019820" (at 264.16 80.01 0)
       (effects (font (size 1.27 1.27)) hide)
     )
@@
       (effects (font (size 1.27 1.27)))
     )
-    (property "Footprint" "Button_Switch_SMD:SW_SPST_B3U-3000P" (at 264.16 115.57 0)
+    (property "Footprint" "Custom:435451019820" (at 264.16 115.57 0)
       (effects (font (size 1.27 1.27)) hide)
     )
@@
       (effects (font (size 1.27 1.27)))
     )
-    (property "Footprint" "Button_Switch_SMD:SW_SPST_B3U-3000P" (at 264.16 88.9 0)
+    (property "Footprint" "Custom:435451019820" (at 264.16 88.9 0)
       (effects (font (size 1.27 1.27)) hide)
     )
@@
     (in_bom yes) (on_board yes) (dnp no) (fields_autoplaced)
     (property "Reference" "C812" (at 205.74 36.2013 0)
-      (effects (font (size 1.27 1.27)) (justify left) hide)
+      (effects (font (size 1.27 1.27)) (justify left))
     )
     (property "Value" "100n" (at 205.74 38.7413 0)
-      (effects (font (size 1.27 1.27)) (justify left) hide)
+      (effects (font (size 1.27 1.27)) (justify left))
     )
     (property "Footprint" "Capacitor_SMD:C_0402_1005Metric_Pad0.74x0.62mm_HandSolder" (at 203.2 36.83 0)
@@
       (effects (font (size 1.27 1.27)))
     )
-    (property "Footprint" "Button_Switch_SMD:SW_SPST_B3U-3000P" (at 264.16 106.68 0)
-      (effects (font (size 1.27 1.27)) hide)
-    )
+    (property "Footprint" "Custom:435451019820" (at 264.16 106.68 0)
+      (effects (font (size 1.27 1.27)) hide)
+    )

Commit message: change pcb
Other:
- note added: "Connector for Encodeur (button)"
- note removed: "Connector for Encodeur"
Changed lines of the file:
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@@
     (effects (font (size 1.27 1.27)) (justify left bottom))
   )
-  (text "Connector for Encodeur" (at 144.78 129.54 0)
+  (text "Connector for Encodeur (button)" (at 144.78 129.54 0)
     (effects (font (size 1.27 1.27)) (justify left bottom))
   )

Commit message: v0 PCB
Connections:
- net ENC_A: now also U801.8 (PC0); no longer J802.3 (Pin_3), U801.20 (PA6)
- net ENC_B: now also U801.9 (PC1); no longer J802.4 (Pin_4), U801.21 (PA7)
- net V_Imes: now also U801.26 (PB2); no longer U801.9 (PC1)
- net V_VPh: now also U801.11 (PC3); no longer U801.8 (PC0)
- net ENC_Z: now reaches U801.10 (PC2)
- net ENC_BTN renamed ENC_BTN_P
- new net ENC_BTN_A: J802.3 (Pin_3), U801.20 (PA6)
- new net ENC_BTN_B: J802.4 (Pin_4), U801.21 (PA7)
- no-connect marks 12 -> 9
Changed lines of the file:
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@@
   (no_connect (at 234.95 46.99))
   (no_connect (at 62.23 101.6))
-  (no_connect (at 97.79 93.98))
   (no_connect (at 62.23 106.68))
-  (no_connect (at 62.23 73.66))
   (no_connect (at 97.79 71.12))
   (no_connect (at 176.53 111.76))
-  (no_connect (at 62.23 76.2))
   (no_connect (at 176.53 109.22))
   (no_connect (at 234.95 41.91))
@@
     (effects (font (size 1.27 1.27)) (justify left bottom))
   )
-  (label "ENC_B" (at 168.91 151.13 180) (fields_autoplaced)
+  (label "ENC_BTN_B" (at 168.91 151.13 180) (fields_autoplaced)
     (effects (font (size 1.27 1.27)) (justify right bottom))
   )
@@
     (effects (font (size 1.27 1.27)) (justify left bottom))
   )
-  (label "ENC_BTN" (at 110.49 58.42 180) (fields_autoplaced)
+  (label "ENC_BTN_P" (at 110.49 58.42 180) (fields_autoplaced)
     (effects (font (size 1.27 1.27)) (justify right bottom))
   )
@@
     (effects (font (size 1.27 1.27)) (justify left bottom))
   )
-  (label "ENC_A" (at 168.91 148.59 180) (fields_autoplaced)
+  (label "ENC_BTN_A" (at 168.91 148.59 180) (fields_autoplaced)
     (effects (font (size 1.27 1.27)) (justify right bottom))
   )
@@
     (effects (font (size 1.27 1.27)) (justify left bottom))
   )
-  (label "ENC_B" (at 110.49 63.5 180) (fields_autoplaced)
+  (label "ENC_BTN_B" (at 110.49 63.5 180) (fields_autoplaced)
     (effects (font (size 1.27 1.27)) (justify right bottom))
   )
@@
     (effects (font (size 1.27 1.27)) (justify left bottom))
   )
-  (label "ENC_BTN" (at 168.91 153.67 180) (fields_autoplaced)
+  (label "ENC_BTN_P" (at 168.91 153.67 180) (fields_autoplaced)
     (effects (font (size 1.27 1.27)) (justify right bottom))
   )
@@
     (effects (font (size 1.27 1.27)) (justify right bottom))
   )
-  (label "ENC_A" (at 110.49 60.96 180) (fields_autoplaced)
+  (label "ENC_BTN_A" (at 110.49 60.96 180) (fields_autoplaced)
     (effects (font (size 1.27 1.27)) (justify right bottom))
   )
@@
     (effects (font (size 1.27 1.27)) (justify right))
   )
+  (hierarchical_label "V_VPh" (shape input) (at 62.23 76.2 180) (fields_autoplaced)
+    (effects (font (size 1.27 1.27)) (justify right))
+  )
   (hierarchical_label "ISO_3V3" (shape input) (at 220.98 21.59 180) (fields_autoplaced)
     (effects (font (size 1.27 1.27)) (justify right))
@@
     (effects (font (size 1.27 1.27)) (justify left))
   )
+  (hierarchical_label "ENC_A" (shape input) (at 62.23 68.58 180) (fields_autoplaced)
+    (effects (font (size 1.27 1.27)) (justify right))
+  )
+  (hierarchical_label "V_Imes" (shape input) (at 97.79 93.98 0) (fields_autoplaced)
+    (effects (font (size 1.27 1.27)) (justify left))
+  )
   (hierarchical_label "ISO_GND" (shape input) (at 271.78 120.65 0) (fields_autoplaced)
     (effects (font (size 1.27 1.27)) (justify left))
@@
     (effects (font (size 1.27 1.27)) (justify right))
   )
+  (hierarchical_label "ENC_B" (shape input) (at 62.23 71.12 180) (fields_autoplaced)
+    (effects (font (size 1.27 1.27)) (justify right))
+  )
   (hierarchical_label "ISO_GND" (shape input) (at 160.02 121.92 180) (fields_autoplaced)
     (effects (font (size 1.27 1.27)) (justify right))
   )
-  (hierarchical_label "V_VPh" (shape input) (at 62.23 68.58 180) (fields_autoplaced)
-    (effects (font (size 1.27 1.27)) (justify right))
-  )
-  (hierarchical_label "V_Imes" (shape input) (at 62.23 71.12 180) (fields_autoplaced)
-    (effects (font (size 1.27 1.27)) (justify right))
-  )
   (hierarchical_label "USART1_RX" (shape input) (at 62.23 81.28 180) (fields_autoplaced)
     (effects (font (size 1.27 1.27)) (justify right))
@@
     (effects (font (size 1.27 1.27)) (justify left))
   )
+  (hierarchical_label "ENC_Z" (shape input) (at 62.23 73.66 180) (fields_autoplaced)
+    (effects (font (size 1.27 1.27)) (justify right))
+  )
   (hierarchical_label "I2C_SDA" (shape input) (at 113.03 66.04 0) (fields_autoplaced)

Commit message: update pcb
Parts:
- C801, C802: value 18p -> 22p; footprint Capacitor_SMD:C_0402_1005Metric_Pad0.74x0.62mm_HandSolder -> Capacitor_SMD:C_0402_1005Metric; Fournisseur (none) -> Wurth; MFR (none) -> 885 012 005 009
- C803, C806, C813: footprint Capacitor_SMD:C_0603_1608Metric_Pad1.08x0.95mm_HandSolder -> Capacitor_SMD:C_0603_1608Metric; Fournisseur (none) -> Wurth; MFR (none) -> 885 012 106 006
- C804, C807, C808, C809, C810, C811, C812, C814, C815, C816, C817, C818: footprint Capacitor_SMD:C_0402_1005Metric_Pad0.74x0.62mm_HandSolder -> Capacitor_SMD:C_0402_1005Metric; Fournisseur (none) -> Wurth; MFR (none) -> 885 012 105 018
- C805: footprint Capacitor_SMD:C_0402_1005Metric_Pad0.74x0.62mm_HandSolder -> Capacitor_SMD:C_0402_1005Metric; Fournisseur (none) -> Wurth; MFR (none) -> 885 012 105 012
- D801, D802, D803, D804: value LED -> Blue LED; footprint LED_SMD:LED_0603_1608Metric_Pad1.05x0.95mm_HandSolder -> LED_SMD:LED_0603_1608Metric; Fournisseur (none) -> Wurth; MFR (none) -> 150 060 BS5 504 0
- J801: Fournisseur (none) -> Wurth; MFR (none) -> 629 722 000 214
- J802, J803, J804: Fournisseur (none) -> Stock
- L801: footprint Inductor_SMD:L_0603_1608Metric_Pad1.05x0.95mm_HandSolder -> Inductor_SMD:L_0603_1608Metric; Fournisseur (none) -> Wurth; MFR (none) -> 744 786 013 9
- R801: footprint Resistor_SMD:R_0402_1005Metric_Pad0.72x0.64mm_HandSolder -> Resistor_SMD:R_0402_1005Metric; Fournisseur (none) -> Farnell; MFR (none) -> MC00625W0402110K; Ref (none) -> 2130433
- R802, R803: footprint Resistor_SMD:R_0402_1005Metric_Pad0.72x0.64mm_HandSolder -> Resistor_SMD:R_0402_1005Metric; Fournisseur (none) -> Sotck
- R804, R805, R806, R807: value 340 -> 390; footprint Resistor_SMD:R_0402_1005Metric_Pad0.72x0.64mm_HandSolder -> Resistor_SMD:R_0402_1005Metric; Fournisseur (none) -> Farnell; MFR (none) -> CRCW0402390RFKEDC; Ref (none) -> 4177482
- SW801, SW802, SW803, SW804, SW805: Fournisseur (none) -> Wurth; MFR (none) -> 435 451 019 820
- U801: Fournisseur (none) -> RS; MFR (none) -> STM32G474RET6; Ref (none) -> 193-9861
- U802: Fournisseur (none) -> RS; MFR (none) -> USBLC6-2SC6; Ref (none) -> 624-7693
- Y801: Fournisseur (none) -> Farnell; MFR (none) -> ABLS-16.000MHZ-20-B-3-H-T; Ref (none) -> 3228387
Connections:
- net USR_LED_1: now also U801.54 (PC12); no longer U801.51 (PA15)
- net USR_LED_2: now also U801.53 (PC11); no longer U801.52 (PC10)
- net USR_LED_3: now also U801.52 (PC10); no longer U801.53 (PC11)
- net USR_LED_4: now also U801.51 (PA15); no longer U801.54 (PC12)
- net Pwr_Enable_U: now reaches U801.2 (PC13)
- net Pwr_Enable_V: now reaches U801.3 (PC14)
- net Pwr_Enable_W: now reaches U801.4 (PC15)
- net Pwr_Enable: no longer names the net of U801.37 (PB15)
- no-connect marks 9 -> 7
