File: Inverter_KiCAD/Vbus_Sense.kicad_sch (KiCad schematic)
At the start: 10 parts

Commit message: update pcb
Parts:
- C?: footprint Capacitor_SMD:C_0402_1005Metric_Pad0.74x0.62mm_HandSolder -> Capacitor_SMD:C_0402_1005Metric; Fournisseur (none) -> Wurth; MFR (none) -> 885 012 205 050
- C? (x3): footprint Capacitor_SMD:C_0402_1005Metric_Pad0.74x0.62mm_HandSolder -> Capacitor_SMD:C_0402_1005Metric; Fournisseur (none) -> Wurth; MFR (none) -> 885 012 205 048
- C? (x2): footprint Capacitor_SMD:C_0402_1005Metric_Pad0.74x0.62mm_HandSolder -> Capacitor_SMD:C_0402_1005Metric; Fournisseur (none) -> Wurth; MFR (none) -> 885 012 105 018
- R?: footprint Resistor_SMD:R_0402_1005Metric_Pad0.72x0.64mm_HandSolder -> Resistor_SMD:R_0402_1005Metric; Fournisseur (none) -> Stock
- R?: footprint Resistor_SMD:R_0402_1005Metric_Pad0.72x0.64mm_HandSolder -> Resistor_SMD:R_0402_1005Metric; Fournisseur (none) -> Farnell; MFR (none) -> MCWR04X1001FTL; Ref (none) -> 2446437
- U?: Fournisseur (none) -> Farnell; MFR (none) -> GO 10-SME/SP3; Ref (none) -> 3796461
- U?: Fournisseur (none) -> RS; MFR (none) -> HCPL-7800A-500E; Ref (none) -> 174-4179
Changed lines of the file:
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@@
       (effects (font (size 1.27 1.27)) (justify left))
     )
-    (property "Footprint" "Capacitor_SMD:C_0402_1005Metric_Pad0.74x0.62mm_HandSolder" (at 121.92 38.1 0)
+    (property "Footprint" "Capacitor_SMD:C_0402_1005Metric" (at 121.92 38.1 0)
       (effects (font (size 1.27 1.27)) hide)
     )
@@
       (effects (font (size 1.27 1.27)) hide)
     )
+    (property "Fournisseur" "Wurth" (at 121.92 38.1 0)
+      (effects (font (size 1.27 1.27)) hide)
+    )
+    (property "MFR" "885 012 205 050" (at 121.92 38.1 0)
+      (effects (font (size 1.27 1.27)) hide)
+    )
     (pin "1")
     (pin "2")
@@
       (effects (font (size 1.27 1.27)) (justify left))
     )
-    (property "Footprint" "Capacitor_SMD:C_0402_1005Metric_Pad0.74x0.62mm_HandSolder" (at 60.96 67.31 0)
+    (property "Footprint" "Capacitor_SMD:C_0402_1005Metric" (at 60.96 67.31 0)
       (effects (font (size 1.27 1.27)) hide)
     )
@@
       (effects (font (size 1.27 1.27)) hide)
     )
+    (property "Fournisseur" "Wurth" (at 60.96 67.31 0)
+      (effects (font (size 1.27 1.27)) hide)
+    )
+    (property "MFR" "885 012 205 048" (at 60.96 67.31 0)
+      (effects (font (size 1.27 1.27)) hide)
+    )
     (pin "1")
     (pin "2")
@@
       (effects (font (size 1.27 1.27)) (justify left))
     )
-    (property "Footprint" "Resistor_SMD:R_0402_1005Metric_Pad0.72x0.64mm_HandSolder" (at 109.22 29.21 0)
+    (property "Footprint" "Resistor_SMD:R_0402_1005Metric" (at 109.22 29.21 0)
       (effects (font (size 1.27 1.27)) hide)
     )
@@
       (effects (font (size 1.27 1.27)) hide)
     )
+    (property "Fournisseur" "Stock" (at 109.22 29.21 0)
+      (effects (font (size 1.27 1.27)) hide)
+    )
     (pin "1")
     (pin "2")
@@
       (effects (font (size 1.27 1.27)) (justify left))
     )
-    (property "Footprint" "Capacitor_SMD:C_0402_1005Metric_Pad0.74x0.62mm_HandSolder" (at 180.34 31.75 0)
+    (property "Footprint" "Capacitor_SMD:C_0402_1005Metric" (at 180.34 31.75 0)
       (effects (font (size 1.27 1.27)) hide)
     )
@@
       (effects (font (size 1.27 1.27)) hide)
     )
+    (property "Fournisseur" "Wurth" (at 180.34 31.75 0)
+      (effects (font (size 1.27 1.27)) hide)
+    )
+    (property "MFR" "885 012 105 018" (at 180.34 31.75 0)
+      (effects (font (size 1.27 1.27)) hide)
+    )
     (pin "1")
     (pin "2")
@@
       (effects (font (size 1.27 1.27)) (justify left))
     )
-    (property "Footprint" "Resistor_SMD:R_0402_1005Metric_Pad0.72x0.64mm_HandSolder" (at 109.22 36.83 0)
+    (property "Footprint" "Resistor_SMD:R_0402_1005Metric" (at 109.22 36.83 0)
       (effects (font (size 1.27 1.27)) hide)
     )
@@
       (effects (font (size 1.27 1.27)) hide)
     )
+    (property "Fournisseur" "Farnell" (at 109.22 36.83 0)
+      (effects (font (size 1.27 1.27)) hide)
+    )
+    (property "MFR" "MCWR04X1001FTL" (at 109.22 36.83 0)
+      (effects (font (size 1.27 1.27)) hide)
+    )
+    (property "Ref" "2446437" (at 109.22 36.83 0)
+      (effects (font (size 1.27 1.27)) hide)
+    )
     (pin "1")
     (pin "2")
@@
       (effects (font (size 1.27 1.27)) (justify left))
     )
-    (property "Footprint" "Capacitor_SMD:C_0402_1005Metric_Pad0.74x0.62mm_HandSolder" (at 52.07 67.31 0)
+    (property "Footprint" "Capacitor_SMD:C_0402_1005Metric" (at 52.07 67.31 0)
       (effects (font (size 1.27 1.27)) hide)
     )
     (property "Datasheet" "~" (at 52.07 67.31 0)
+      (effects (font (size 1.27 1.27)) hide)
+    )
+    (property "Fournisseur" "Wurth" (at 52.07 67.31 0)
+      (effects (font (size 1.27 1.27)) hide)
+    )
+    (property "MFR" "885 012 205 048" (at 52.07 67.31 0)
       (effects (font (size 1.27 1.27)) hide)
     )
@@
     (property "Datasheet" "GO 10-SME" (at 46.99 24.13 0)
       (effects (font (size 1.27 1.27) italic) hide)
+    )
+    (property "MFR" "GO 10-SME/SP3" (at 52.07 41.91 0)
+      (effects (font (size 1.27 1.27)) hide)
+    )
+    (property "Fournisseur" "Farnell" (at 52.07 41.91 0)
+      (effects (font (size 1.27 1.27)) hide)
+    )
+    (property "Ref" "3796461" (at 52.07 41.91 0)
+      (effects (font (size 1.27 1.27)) hide)
     )
     (pin "1")
@@
       (effects (font (size 1.27 1.27)) (justify left))
     )
-    (property "Footprint" "Capacitor_SMD:C_0402_1005Metric_Pad0.74x0.62mm_HandSolder" (at 190.5 31.75 0)
+    (property "Footprint" "Capacitor_SMD:C_0402_1005Metric" (at 190.5 31.75 0)
       (effects (font (size 1.27 1.27)) hide)
     )
@@
       (effects (font (size 1.27 1.27)) hide)
     )
+    (property "Fournisseur" "Wurth" (at 190.5 31.75 0)
+      (effects (font (size 1.27 1.27)) hide)
+    )
+    (property "MFR" "885 012 105 018" (at 190.5 31.75 0)
+      (effects (font (size 1.27 1.27)) hide)
+    )
     (pin "1")
     (pin "2")
@@
       (effects (font (size 1.27 1.27)) (justify left))
     )
-    (property "Footprint" "Capacitor_SMD:C_0402_1005Metric_Pad0.74x0.62mm_HandSolder" (at 41.91 67.31 0)
+    (property "Footprint" "Capacitor_SMD:C_0402_1005Metric" (at 41.91 67.31 0)
       (effects (font (size 1.27 1.27)) hide)
     )
     (property "Datasheet" "~" (at 41.91 67.31 0)
+      (effects (font (size 1.27 1.27)) hide)
+    )
+    (property "Fournisseur" "Wurth" (at 41.91 67.31 0)
+      (effects (font (size 1.27 1.27)) hide)
+    )
+    (property "MFR" "885 012 205 048" (at 41.91 67.31 0)
       (effects (font (size 1.27 1.27)) hide)
     )
@@
       (effects (font (size 1.27 1.27) italic) hide)
     )
-    (pin "1")
+    (property "Fournisseur" "RS" (at 146.05 34.29 0)
+      (effects (font (size 1.27 1.27)) hide)
+    )
+    (property "MFR" "HCPL-7800A-500E" (at 146.05 34.29 0)
+      (effects (font (size 1.27 1.27)) hide)
+    )
+    (property "Ref" "174-4179" (at 146.05 34.29 0)
+      (effects (font (size 1.27 1.27)) hide)
+    )
+    (pin "1")
