File: Inverter_KiCAD/Vbus_Sense.kicad_sch (KiCad schematic)
At the start: 10 parts

Commit message: update pcb
Parts:
- R?: value 160k -> 470k
Other:
- note added: "HCPL-7800A Gain : 8V/V (differential) 4V/V (signe ended) Offset : 2.5V"
- note removed: "HCPL-7800A Gain : 8V/V"
Changed lines of the file:
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@@
     (fill (type none))
+  )
+  (text "HCPL-7800A Gain :\n	8V/V (differential)\n	4V/V (signe ended)\nOffset : 2.5V"
+    (at 157.48 22.86 0)
+    (effects (font (size 1.27 1.27)) (justify left bottom))
   )
   (text "Hall current" (at 16.51 17.78 0)
@@
   )
   (text "Vin+ max value : 0.41V" (at 111.76 25.4 0)
-    (effects (font (size 1.27 1.27)) (justify left bottom))
-  )
-  (text "HCPL-7800A Gain : 8V/V" (at 134.62 20.32 0)
     (effects (font (size 1.27 1.27)) (justify left bottom))
   )
@@
   (symbol (lib_id "Device:R_Small") (at 109.22 29.21 0) (unit 1)
     (in_bom yes) (on_board yes) (dnp no) (fields_autoplaced)
-    (property "Reference" "R?" (at 111.76 28.575 0)
+    (property "Reference" "R?" (at 111.76 27.94 0)
       (effects (font (size 1.27 1.27)) (justify left))
     )
-    (property "Value" "160k" (at 111.76 31.115 0)
+    (property "Value" "470k" (at 111.76 30.48 0)
       (effects (font (size 1.27 1.27)) (justify left))
     )
