File: Inverter_KiCAD/break.kicad_sch (KiCad schematic)
At the start: 14 parts, among them J901 Conn_01x02, Q901 BUK9637-100E, U901 ACPL-077L, U902 TC1412

Commit message: v0 PCB
Parts:
- removed J901: Conn_01x02, Custom:691311700002, symbol Connector_Generic:Conn_01x02
- added J902: Conn_01x02, Custom:691311500102, symbol Connector_Generic:Conn_01x02
Connections:
- net Break_Drain_Mosfet: now also J902.1 (Pin_1)
- net VSupply_AB: now also J902.2 (Pin_2)
Other:
- note removed: "nouvelle ref : 691311500102"
Changed lines of the file:
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@@
     (stroke (width 0) (type default))
   )
-  (wire (pts (xy 168.91 30.48) (xy 176.53 30.48))
+  (wire (pts (xy 168.91 30.48) (xy 182.88 30.48))
     (stroke (width 0) (type default))
   )
@@
     (effects (font (size 1.27 1.27)) (justify left bottom))
   )
-  (text "nouvelle ref : \n691311500102" (at 175.26 26.67 0)
-    (effects (font (size 3.4 3.4) (thickness 0.68) bold) (justify left bottom))
-  )
   (text "For resistance :\n5 ohm / 100W" (at 175.26 45.72 0)
     (effects (font (size 1.27 1.27)) (justify left bottom))
@@
     (effects (font (size 1.27 1.27)) (justify right))
   )
-  (hierarchical_label "VSupply_AB" (shape input) (at 176.53 30.48 0) (fields_autoplaced)
+  (hierarchical_label "VSupply_AB" (shape input) (at 182.88 30.48 0) (fields_autoplaced)
     (effects (font (size 1.27 1.27)) (justify left))
   )
@@
       (effects (font (size 1.27 1.27)) hide)
     )
-    (property "Datasheet" "~" (at 160.02 30.48 0)
+    (property "Datasheet" "https://www.vishay.com/docs/94927/vs-15tq060s-m3.pdf" (at 160.02 30.48 0)
       (effects (font (size 1.27 1.27)) hide)
     )
@@
       (effects (font (size 1.27 1.27)) hide)
     )
-    (property "Datasheet" "~" (at 165.1 36.83 0)
+    (property "Datasheet" "https://www.vishay.com/docs/94927/vs-15tq060s-m3.pdf" (at 165.1 36.83 0)
       (effects (font (size 1.27 1.27)) hide)
     )
@@
         (path "/5e6c1e3f-0815-454a-8acb-8e3e2d064875/63722f1b-78db-4d3b-ade4-7dd7cc6c956f"
           (reference "D1") (unit 1)
-        )
-      )
-    )
-  )
-  (symbol (lib_id "Connector_Generic:Conn_01x02") (at 175.26 38.1 0) (mirror x) (unit 1)
-    (in_bom yes) (on_board yes) (dnp no)
-    (property "Reference" "J901" (at 175.26 30.48 0)
-      (effects (font (size 1.27 1.27)))
-    )
-    (property "Value" "Conn_01x02" (at 175.26 33.02 0)
-      (effects (font (size 1.27 1.27)))
-    )
-    (property "Footprint" "Custom:691311700002" (at 175.26 38.1 0)
-      (effects (font (size 1.27 1.27)) hide)
-    )
-    (property "Datasheet" "https://www.we-online.com/components/products/datasheet/691311700002.pdf" (at 175.26 38.1 0)
-      (effects (font (size 1.27 1.27)) hide)
-    )
-    (property "MFR" "691311700002" (at 175.26 38.1 0)
-      (effects (font (size 1.27 1.27)) hide)
-    )
-    (property "Field5" "" (at 175.26 38.1 0)
-      (effects (font (size 1.27 1.27)) hide)
-    )
-    (pin "1")
-    (pin "2")
-    (instances
-      (project "Inverter_KiCAD"
-        (path "/5e6c1e3f-0815-454a-8acb-8e3e2d064875/63722f1b-78db-4d3b-ade4-7dd7cc6c956f"
-          (reference "J901") (unit 1)
         )
       )
@@
         )
       )
+    )
+  )
+  (symbol (lib_id "Connector_Generic:Conn_01x02") (at 175.26 38.1 0) (mirror x) (unit 1)
+    (in_bom yes) (on_board yes) (dnp no)
+    (property "Reference" "J902" (at 175.26 30.48 0)
+      (effects (font (size 1.27 1.27)))
+    )
+    (property "Value" "Conn_01x02" (at 175.26 33.02 0)
+      (effects (font (size 1.27 1.27)))
+    )
+    (property "Footprint" "Custom:691311500102" (at 175.26 38.1 0)
+      (effects (font (size 1.27 1.27)) hide)
+    )
+    (property "Datasheet" "https://www.we-online.com/components/products/datasheet/691311500102.pdf" (at 175.26 38.1 0)
+      (effects (font (size 1.27 1.27)) hide)
+    )
+    (property "MFR" "691311700102" (at 175.26 38.1 0)
+      (effects (font (size 1.27 1.27)) hide)
+    )
+    (property "Field5" "" (at 175.26 38.1 0)
+      (effects (font (size 1.27 1.27)) hide)
+    )
+    (pin "1")
+    (pin "2")
+    (instances
+      (project "Inverter_KiCAD"
+        (path "/5e6c1e3f-0815-454a-8acb-8e3e2d064875/63722f1b-78db-4d3b-ade4-7dd7cc6c956f"
+          (reference "J902") (unit 1)
+        )
+        (path "/5e6c1e3f-0815-454a-8acb-8e3e2d064875"
+          (reference "J1") (unit 1)
+        )
+      )

Commit message: update pcb
Parts:
- C901, C902: footprint Capacitor_SMD:C_0402_1005Metric_Pad0.74x0.62mm_HandSolder -> Capacitor_SMD:C_0402_1005Metric; Fournisseur (none) -> Wurth; MFR (none) -> 885 012 105 018
- C903: footprint Capacitor_SMD:C_0402_1005Metric_Pad0.74x0.62mm_HandSolder -> Capacitor_SMD:C_0402_1005Metric; Fournisseur (none) -> Wurth; MFR (none) -> 885 012 105 012
- C904: footprint Capacitor_SMD:C_0402_1005Metric_Pad0.74x0.62mm_HandSolder -> Capacitor_SMD:C_0402_1005Metric; Fournisseur (none) -> Wurth; MFR (none) -> 885 012 205 044
- D901: value Red -> Red LED; footprint LED_SMD:LED_0603_1608Metric_Pad1.05x0.95mm_HandSolder -> LED_SMD:LED_0603_1608Metric; Fournisseur (none) -> Wurth; MFR (none) -> 150 060 RS5 504 0
- D902: Fournisseur (none) -> Farnell; MFR (none) -> VS-15TQ060S-M3; Ref (none) -> 2909608
- D903: renamed from D1; Fournisseur (none) -> Farnell; MFR (none) -> VS-15TQ060S-M3; Ref (none) -> 2909608
- J901: renamed from J902; Fournisseur (none) -> Wurth; MFR 691311700102 -> 691 311 700 102
- Q901: Fournisseur (none) -> Farnell; MFR (none) -> BUK9637-100E,118; Ref (none) -> 2254193
- R901: value 100 -> 390; footprint Resistor_SMD:R_0402_1005Metric_Pad0.72x0.64mm_HandSolder -> Resistor_SMD:R_0402_1005Metric; Fournisseur (none) -> Farnell; MFR (none) -> CRCW0402390RFKEDC; Ref (none) -> 4177482
- R902: footprint Resistor_SMD:R_0402_1005Metric_Pad0.72x0.64mm_HandSolder -> Resistor_SMD:R_0402_1005Metric; Fournisseur (none) -> Farnell; MFR (none) -> MC00625W0402110K; Ref (none) -> 2130433
- R903: value 5 -> 4.7; footprint Resistor_SMD:R_1206_3216Metric_Pad1.30x1.75mm_HandSolder -> Resistor_SMD:R_1206_3216Metric; Fournisseur (none) -> Stock
- U901: Fournisseur (none) -> RS; MFR (none) -> ACPL-077L-500E; Ref (none) -> 230-5293
- U902: Fournisseur (none) -> RS; MFR (none) -> TC1412NEOA; Ref (none) -> 1834898
Changed lines of the file:
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@@
+      (effects (font (size 1.27 1.27)) hide)
+    )
+    (property "Fournisseur" "RS" (at 104.14 30.48 0)
+      (effects (font (size 1.27 1.27)) hide)
+    )
+    (property "MFR" "TC1412NEOA" (at 104.14 30.48 0)
+      (effects (font (size 1.27 1.27)) hide)
+    )
+    (property "Ref" "1834898" (at 104.14 30.48 0)
       (effects (font (size 1.27 1.27)) hide)
     )
@@
       (effects (font (size 1.27 1.27)))
     )
-    (property "Value" "5" (at 157.48 50.8 90)
-      (effects (font (size 1.27 1.27)))
-    )
-    (property "Footprint" "Resistor_SMD:R_1206_3216Metric_Pad1.30x1.75mm_HandSolder" (at 157.48 53.34 0)
+    (property "Value" "4.7" (at 157.48 50.8 90)
+      (effects (font (size 1.27 1.27)))
+    )
+    (property "Footprint" "Resistor_SMD:R_1206_3216Metric" (at 157.48 53.34 0)
       (effects (font (size 1.27 1.27)) hide)
     )
@@
       (effects (font (size 1.27 1.27)) hide)
     )
+    (property "Fournisseur" "Stock" (at 157.48 53.34 0)
+      (effects (font (size 1.27 1.27)) hide)
+    )
     (pin "1")
     (pin "2")
@@
       (effects (font (size 1.27 1.27)) (justify left))
     )
-    (property "Footprint" "Capacitor_SMD:C_0402_1005Metric_Pad0.74x0.62mm_HandSolder" (at 100.33 54.61 0)
+    (property "Footprint" "Capacitor_SMD:C_0402_1005Metric" (at 100.33 54.61 0)
       (effects (font (size 1.27 1.27)) hide)
     )
@@
       (effects (font (size 1.27 1.27)) hide)
     )
+    (property "Fournisseur" "Wurth" (at 100.33 54.61 0)
+      (effects (font (size 1.27 1.27)) hide)
+    )
+    (property "MFR" "885 012 105 012" (at 100.33 54.61 0)
+      (effects (font (size 1.27 1.27)) hide)
+    )
     (pin "1")
     (pin "2")
@@
       (effects (font (size 1.27 1.27)) (justify left))
     )
-    (property "Footprint" "Capacitor_SMD:C_0402_1005Metric_Pad0.74x0.62mm_HandSolder" (at 53.34 54.61 0)
+    (property "Footprint" "Capacitor_SMD:C_0402_1005Metric" (at 53.34 54.61 0)
       (effects (font (size 1.27 1.27)) hide)
     )
@@
       (effects (font (size 1.27 1.27)) hide)
     )
+    (property "Fournisseur" "Wurth" (at 53.34 54.61 0)
+      (effects (font (size 1.27 1.27)) hide)
+    )
+    (property "MFR" "885 012 105 018" (at 53.34 54.61 0)
+      (effects (font (size 1.27 1.27)) hide)
+    )
     (pin "1")
     (pin "2")
@@
     )
     (property "Datasheet" "https://www.vishay.com/docs/94927/vs-15tq060s-m3.pdf" (at 160.02 30.48 0)
+      (effects (font (size 1.27 1.27)) hide)
+    )
+    (property "Fournisseur" "Farnell" (at 160.02 30.48 0)
+      (effects (font (size 1.27 1.27)) hide)
+    )
+    (property "MFR" "VS-15TQ060S-M3" (at 160.02 30.48 0)
+      (effects (font (size 1.27 1.27)) hide)
+    )
+    (property "Ref" "2909608" (at 160.02 30.48 0)
       (effects (font (size 1.27 1.27)) hide)
     )
@@
   (symbol (lib_id "Device:D_Schottky") (at 165.1 36.83 270) (unit 1)
     (in_bom yes) (on_board yes) (dnp no)
-    (property "Reference" "D1" (at 160.02 35.56 90)
+    (property "Reference" "D903" (at 160.02 35.56 90)
       (effects (font (size 1.27 1.27)) (justify left))
     )
@@
       (effects (font (size 1.27 1.27)) hide)
     )
+    (property "Fournisseur" "Farnell" (at 165.1 36.83 0)
+      (effects (font (size 1.27 1.27)) hide)
+    )
+    (property "MFR" "VS-15TQ060S-M3" (at 165.1 36.83 0)
+      (effects (font (size 1.27 1.27)) hide)
+    )
+    (property "Ref" "2909608" (at 165.1 36.83 0)
+      (effects (font (size 1.27 1.27)) hide)
+    )
     (pin "2")
     (pin "3")
@@
       (project "Inverter_KiCAD"
         (path "/5e6c1e3f-0815-454a-8acb-8e3e2d064875/63722f1b-78db-4d3b-ade4-7dd7cc6c956f"
-          (reference "D1") (unit 1)
+          (reference "D903") (unit 1)
         )
       )
@@
   (symbol (lib_id "Device:LED_Small") (at 40.64 53.34 90) (unit 1)
     (in_bom yes) (on_board yes) (dnp no) (fields_autoplaced)
-    (property "Reference" "D901" (at 43.18 52.6415 90)
+    (property "Reference" "D901" (at 43.18 52.0065 90)
       (effects (font (size 1.27 1.27)) (justify right))
     )
-    (property "Value" "Red" (at 43.18 55.1815 90)
+    (property "Value" "Red LED" (at 43.18 54.5465 90)
       (effects (font (size 1.27 1.27)) (justify right))
     )
-    (property "Footprint" "LED_SMD:LED_0603_1608Metric_Pad1.05x0.95mm_HandSolder" (at 40.64 53.34 90)
+    (property "Footprint" "LED_SMD:LED_0603_1608Metric" (at 40.64 53.34 90)
       (effects (font (size 1.27 1.27)) hide)
     )
     (property "Datasheet" "~" (at 40.64 53.34 90)
+      (effects (font (size 1.27 1.27)) hide)
+    )
+    (property "Fournisseur" "Wurth" (at 40.64 53.34 0)
+      (effects (font (size 1.27 1.27)) hide)
+    )
+    (property "MFR" "150 060 RS5 504 0" (at 40.64 53.34 0)
       (effects (font (size 1.27 1.27)) hide)
     )
@@
       (effects (font (size 1.27 1.27)) (justify left))
     )
-    (property "Footprint" "Resistor_SMD:R_0402_1005Metric_Pad0.72x0.64mm_HandSolder" (at 88.9 31.75 0)
+    (property "Footprint" "Resistor_SMD:R_0402_1005Metric" (at 88.9 31.75 0)
       (effects (font (size 1.27 1.27)) hide)
     )
@@
       (effects (font (size 1.27 1.27)) hide)
     )
+    (property "Fournisseur" "Farnell" (at 88.9 31.75 0)
+      (effects (font (size 1.27 1.27)) hide)
+    )
+    (property "MFR" "MC00625W0402110K" (at 88.9 31.75 0)
+      (effects (font (size 1.27 1.27)) hide)
+    )
+    (property "Ref" "2130433" (at 88.9 31.75 0)
+      (effects (font (size 1.27 1.27)) hide)
+    )
     (pin "1")
     (pin "2")
@@
     )
     (property "Datasheet" "" (at 38.1 30.48 0)
+      (effects (font (size 1.27 1.27)) hide)
+    )
+    (property "Fournisseur" "RS" (at 44.45 34.29 0)
+      (effects (font (size 1.27 1.27)) hide)
+    )
+    (property "MFR" "ACPL-077L-500E" (at 44.45 34.29 0)
+      (effects (font (size 1.27 1.27)) hide)
+    )
+    (property "Ref" "230-5293" (at 44.45 34.29 0)
       (effects (font (size 1.27 1.27)) hide)
     )
@@
       (effects (font (size 1.27 1.27)) (justify left) hide)
     )
+    (property "Ref" "2254193" (at 166.37 53.34 0)
+      (effects (font (size 1.27 1.27)) hide)
+    )
+    (property "Fournisseur" "Farnell" (at 166.37 53.34 0)
+      (effects (font (size 1.27 1.27)) hide)
+    )
+    (property "MFR" "BUK9637-100E,118" (at 166.37 53.34 0)
+      (effects (font (size 1.27 1.27)) hide)
+    )
     (pin "1")
     (pin "2")
@@
       (effects (font (size 1.27 1.27)) (justify left))
     )
-    (property "Footprint" "Capacitor_SMD:C_0402_1005Metric_Pad0.74x0.62mm_HandSolder" (at 109.22 54.61 0)
+    (property "Footprint" "Capacitor_SMD:C_0402_1005Metric" (at 109.22 54.61 0)
       (effects (font (size 1.27 1.27)) hide)
     )
     (property "Datasheet" "~" (at 109.22 54.61 0)
+      (effects (font (size 1.27 1.27)) hide)
+    )
+    (property "Fournisseur" "Wurth" (at 109.22 54.61 0)
+      (effects (font (size 1.27 1.27)) hide)
+    )
+    (property "MFR" "885 012 205 044" (at 109.22 54.61 0)
       (effects (font (size 1.27 1.27)) hide)
     )
@@
   (symbol (lib_id "Connector_Generic:Conn_01x02") (at 175.26 38.1 0) (mirror x) (unit 1)
     (in_bom yes) (on_board yes) (dnp no)
-    (property "Reference" "J902" (at 175.26 30.48 0)
+    (property "Reference" "J901" (at 175.26 30.48 0)
       (effects (font (size 1.27 1.27)))
     )
@@
       (effects (font (size 1.27 1.27)) hide)
     )
-    (property "MFR" "691311700102" (at 175.26 38.1 0)
+    (property "MFR" "691 311 700 102" (at 175.26 38.1 0)
       (effects (font (size 1.27 1.27)) hide)
     )
@@
       (effects (font (size 1.27 1.27)) hide)
     )
-    (pin "1")
-    (pin "2")
-    (instances
-      (project "Inverter_KiCAD"
-        (path "/5e6c1e3f-0815-454a-8acb-8e3e2d064875/63722f1b-78db-4d3b-ade4-7dd7cc6c956f"
-          (reference "J902") (unit 1)
+    (property "Fournisseur" "Wurth" (at 175.26 38.1 0)
+      (effects (font (size 1.27 1.27)) hide)
+    )
+    (pin "1")
+    (pin "2")
+    (instances
+      (project "Inverter_KiCAD"
+        (path "/5e6c1e3f-0815-454a-8acb-8e3e2d064875/63722f1b-78db-4d3b-ade4-7dd7cc6c956f"
+          (reference "J901") (unit 1)
         )
         (path "/5e6c1e3f-0815-454a-8acb-8e3e2d064875"
@@
       (effects (font (size 1.27 1.27)))
     )
-    (property "Value" "100" (at 36.83 46.99 90)
-      (effects (font (size 1.27 1.27)))
-    )
-    (property "Footprint" "Resistor_SMD:R_0402_1005Metric_Pad0.72x0.64mm_HandSolder" (at 36.83 49.53 0)
+    (property "Value" "390" (at 36.83 46.99 90)
+      (effects (font (size 1.27 1.27)))
+    )
+    (property "Footprint" "Resistor_SMD:R_0402_1005Metric" (at 36.83 49.53 0)
       (effects (font (size 1.27 1.27)) hide)
     )
@@
       (effects (font (size 1.27 1.27)) hide)
     )
+    (property "Fournisseur" "Farnell" (at 36.83 49.53 0)
+      (effects (font (size 1.27 1.27)) hide)
+    )
+    (property "MFR" "CRCW0402390RFKEDC" (at 36.83 49.53 0)
+      (effects (font (size 1.27 1.27)) hide)
+    )
+    (property "Ref" "4177482" (at 36.83 49.53 0)
+      (effects (font (size 1.27 1.27)) hide)
+    )
     (pin "1")
     (pin "2")
@@
       (effects (font (size 1.27 1.27)) (justify left))
     )
-    (property "Footprint" "Capacitor_SMD:C_0402_1005Metric_Pad0.74x0.62mm_HandSolder" (at 62.23 54.61 0)
+    (property "Footprint" "Capacitor_SMD:C_0402_1005Metric" (at 62.23 54.61 0)
       (effects (font (size 1.27 1.27)) hide)
     )
@@
       (effects (font (size 1.27 1.27)) hide)
     )
+    (property "Fournisseur" "Wurth" (at 62.23 54.61 0)
+      (effects (font (size 1.27 1.27)) hide)
+    )
+    (property "MFR" "885 012 105 018" (at 62.23 54.61 0)
+      (effects (font (size 1.27 1.27)) hide)
+    )
