File: Inverter_KiCAD/tempSensor.kicad_sch (KiCad schematic)
At the start: 3 parts, among them U1201 TCN75A

Commit message: update pcb
Parts:
- C1201: footprint Capacitor_SMD:C_0402_1005Metric_Pad0.74x0.62mm_HandSolder -> Capacitor_SMD:C_0402_1005Metric; Fournisseur (none) -> Wurth; MFR (none) -> 885 012 105 018
- R1201: footprint Resistor_SMD:R_0402_1005Metric_Pad0.72x0.64mm_HandSolder -> Resistor_SMD:R_0402_1005Metric; Fournisseur (none) -> Stock
- U1201: Fournisseur (none) -> RS; MFR (none) -> TCN75AVOA; Ref (none) -> 738-6014
Changed lines of the file:
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@@
       (effects (font (size 1.27 1.27)) (justify left))
     )
-    (property "Footprint" "Capacitor_SMD:C_0402_1005Metric_Pad0.74x0.62mm_HandSolder" (at 88.9 35.56 0)
+    (property "Footprint" "Capacitor_SMD:C_0402_1005Metric" (at 88.9 35.56 0)
       (effects (font (size 1.27 1.27)) hide)
     )
     (property "Datasheet" "~" (at 88.9 35.56 0)
+      (effects (font (size 1.27 1.27)) hide)
+    )
+    (property "Fournisseur" "Wurth" (at 88.9 35.56 0)
+      (effects (font (size 1.27 1.27)) hide)
+    )
+    (property "MFR" "885 012 105 018" (at 88.9 35.56 0)
       (effects (font (size 1.27 1.27)) hide)
     )
@@
       (effects (font (size 1.27 1.27)) hide)
     )
+    (property "Fournisseur" "RS" (at 40.64 29.21 0)
+      (effects (font (size 1.27 1.27)) hide)
+    )
+    (property "MFR" "TCN75AVOA" (at 40.64 29.21 0)
+      (effects (font (size 1.27 1.27)) hide)
+    )
+    (property "Ref" "738-6014" (at 40.64 29.21 0)
+      (effects (font (size 1.27 1.27)) hide)
+    )
     (pin "1")
     (pin "2")
@@
       (effects (font (size 1.27 1.27)))
     )
-    (property "Footprint" "Resistor_SMD:R_0402_1005Metric_Pad0.72x0.64mm_HandSolder" (at 55.88 27.94 0)
+    (property "Footprint" "Resistor_SMD:R_0402_1005Metric" (at 55.88 27.94 0)
       (effects (font (size 1.27 1.27)) hide)
     )
@@
       (effects (font (size 1.27 1.27)) hide)
     )
+    (property "Fournisseur" "Stock" (at 55.88 27.94 0)
+      (effects (font (size 1.27 1.27)) hide)
+    )
