File: Inverter_KiCAD/Arm_IRF540NBbF.kicad_sch (KiCad schematic)
At the start: 23 parts, among them Q201 HCPL-315J-500E, Q202 IRF540N, Q203 IRF540N, U201 MPRB2415S-6W, U202 MPRB2415S-6W, U203 HCPL-7800A, U204 GO 10-SME/SP3

Commit message: rooting done
Parts:
- removed U203: HCPL-7800A, Custom:HCPL-7800A, symbol Custom:HCPL-7800A
- added U303: HCPL-7800-500E, Custom:DIP-8 Gull Wing, symbol Custom:HCPL-7800-500E
Connections:
- net 5V: now also U303.1 (VDD1)
- net GND: now also U303.3 (VIN-), U303.4 (GND1)
- net ISO_5V: now also U303.8 (VDD2)
- net ISO_GND: now also U303.5 (GND2), U303.6 (VOUT-)
- net VPH_Sense: now also U303.7 (VOUT+)
- net at C205.1, R205.2, R206.1: now also U303.2 (VIN+)
Changed lines of the file:
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@@
+    )
+  )
+  (symbol (lib_id "Custom:HCPL-7800-500E") (at 162.56 106.68 0) (unit 1)
+    (in_bom yes) (on_board yes) (dnp no) (fields_autoplaced)
+    (property "Reference" "U303" (at 162.56 95.25 0)
+      (effects (font (size 1.524 1.524)))
+    )
+    (property "Value" "HCPL-7800-500E" (at 162.56 97.79 0)
+      (effects (font (size 1.524 1.524)))
+    )
+    (property "Footprint" "Custom:DIP-8 Gull Wing" (at 166.37 121.92 0)
+      (effects (font (size 1.27 1.27) italic) hide)
+    )
+    (property "Datasheet" "" (at 163.83 119.38 0)
+      (effects (font (size 1.27 1.27) italic) hide)
+    )
+    (pin "1")
+    (pin "2")
+    (pin "3")
+    (pin "4")
+    (pin "5")
+    (pin "6")
+    (pin "7")
+    (pin "8")
+    (instances
+      (project "Inverter_KiCAD"
+        (path "/5e6c1e3f-0815-454a-8acb-8e3e2d064875/7e6a23ff-8591-450f-995d-37af863aff63"
+          (reference "U303") (unit 1)
+        )
+        (path "/5e6c1e3f-0815-454a-8acb-8e3e2d064875/9da1d24f-0210-4c44-b691-d03fb3165448"
+          (reference "U203") (unit 1)
+        )
+        (path "/5e6c1e3f-0815-454a-8acb-8e3e2d064875/9544454d-ec1d-4fae-9228-d7a31bd25ddf"
+          (reference "U403") (unit 1)
+        )
+      )
     )
   )
@@
         )
       )
-    )
-  )
-  (symbol (lib_id "Custom:HCPL-7800A") (at 162.56 106.68 0) (unit 1)
-    (in_bom yes) (on_board yes) (dnp no) (fields_autoplaced)
-    (property "Reference" "U203" (at 162.56 95.25 0)
-      (effects (font (size 1.524 1.524)))
-    )
-    (property "Value" "HCPL-7800A" (at 162.56 97.79 0)
-      (effects (font (size 1.524 1.524)))
-    )
-    (property "Footprint" "Custom:HCPL-7800A" (at 166.37 121.92 0)
-      (effects (font (size 1.27 1.27) italic) hide)
-    )
-    (property "Datasheet" "HCPL-7800A" (at 163.83 119.38 0)
-      (effects (font (size 1.27 1.27) italic) hide)
-    )
-    (pin "1")
-    (pin "2")
-    (pin "3")
-    (pin "4")
-    (pin "5")
-    (pin "6")
-    (pin "7")
-    (pin "8")
-    (instances
-      (project "Inverter_KiCAD"
-        (path "/5e6c1e3f-0815-454a-8acb-8e3e2d064875/9da1d24f-0210-4c44-b691-d03fb3165448"
-          (reference "U203") (unit 1)
-        )
-        (path "/5e6c1e3f-0815-454a-8acb-8e3e2d064875/7e6a23ff-8591-450f-995d-37af863aff63"
-          (reference "U303") (unit 1)
-        )
-        (path "/5e6c1e3f-0815-454a-8acb-8e3e2d064875/9544454d-ec1d-4fae-9228-d7a31bd25ddf"
-          (reference "U403") (unit 1)
-        )
-      )

Commit message: v0 PCB
Parts:
- added C1: 10u, Capacitor_SMD:C_0805_2012Metric, symbol Device:C_Small
Connections:
- net GND: now also C1.2
- net Vbus: now also C1.1
Changed lines of the file:
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@@
+    (stroke (width 0) (type default))
+  )
+  (wire (pts (xy 162.56 16.51) (xy 162.56 17.78))
     (stroke (width 0) (type default))
   )
@@
     (stroke (width 0) (type default))
   )
+  (wire (pts (xy 162.56 22.86) (xy 162.56 24.13))
+    (stroke (width 0) (type default))
+  )
   (wire (pts (xy 55.88 128.27) (xy 59.69 128.27))
     (stroke (width 0) (type default))
@@
     (stroke (width 0) (type default))
   )
+  (wire (pts (xy 156.21 24.13) (xy 162.56 24.13))
+    (stroke (width 0) (type default))
+  )
   (wire (pts (xy 82.55 99.06) (xy 88.9 99.06))
+    (stroke (width 0) (type default))
+  )
+  (wire (pts (xy 156.21 16.51) (xy 162.56 16.51))
     (stroke (width 0) (type default))
   )
@@
     (effects (font (size 1.27 1.27)) (justify right))
   )
+  (hierarchical_label "Vbus" (shape input) (at 156.21 16.51 180) (fields_autoplaced)
+    (effects (font (size 1.27 1.27)) (justify right))
+  )
   (hierarchical_label "ISO_15V" (shape input) (at 55.88 128.27 180) (fields_autoplaced)
     (effects (font (size 1.27 1.27)) (justify right))
@@
   )
   (hierarchical_label "GND" (shape input) (at 142.24 67.31 270) (fields_autoplaced)
+    (effects (font (size 1.27 1.27)) (justify right))
+  )
+  (hierarchical_label "GND" (shape input) (at 156.21 24.13 180) (fields_autoplaced)
     (effects (font (size 1.27 1.27)) (justify right))
   )
@@
         )
       )
+    )
+  )
+  (symbol (lib_id "Device:C_Small") (at 162.56 20.32 0) (unit 1)
+    (in_bom yes) (on_board yes) (dnp no) (fields_autoplaced)
+    (property "Reference" "C1" (at 165.1 19.0563 0)
+      (effects (font (size 1.27 1.27)) (justify left))
+    )
+    (property "Value" "10u" (at 165.1 21.5963 0)
+      (effects (font (size 1.27 1.27)) (justify left))
+    )
+    (property "Footprint" "Capacitor_SMD:C_0805_2012Metric" (at 162.56 20.32 0)
+      (effects (font (size 1.27 1.27)) hide)
+    )
+    (property "Datasheet" "~" (at 162.56 20.32 0)
+      (effects (font (size 1.27 1.27)) hide)
+    )
+    (pin "1")
+    (pin "2")
+    (instances
+      (project "Inverter_KiCAD"
+        (path "/5e6c1e3f-0815-454a-8acb-8e3e2d064875/3abd505c-2b96-4cc2-9359-42e0642ca937"
+          (reference "C1") (unit 1)
+        )
+        (path "/5e6c1e3f-0815-454a-8acb-8e3e2d064875/9da1d24f-0210-4c44-b691-d03fb3165448"
+          (reference "C211") (unit 1)
+        )
+        (path "/5e6c1e3f-0815-454a-8acb-8e3e2d064875/7e6a23ff-8591-450f-995d-37af863aff63"
+          (reference "C311") (unit 1)
+        )
+        (path "/5e6c1e3f-0815-454a-8acb-8e3e2d064875/9544454d-ec1d-4fae-9228-d7a31bd25ddf"
+          (reference "C411") (unit 1)
+        )
+      )

Commit message: update pcb
Parts:
- added D804 (x2): Red LED, LED_SMD:LED_0603_1608Metric, symbol Device:LED
- added D804: Green LED, LED_SMD:LED_0603_1608Metric, symbol Device:LED
- added R207, R209: 10k, Resistor_SMD:R_0402_1005Metric, symbol Device:R_Small
- added R807 (x3): 390, Resistor_SMD:R_0402_1005Metric, symbol Device:R_Small
- C1: footprint Capacitor_SMD:C_0805_2012Metric -> Capacitor_SMD:C_2220_5650Metric; Fournisseur (none) -> Wurth; MFR (none) -> 885 012 214 001; URL (none) -> https://www.we-online.com/components/products/datasheet/885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
- C201, C202: Fournisseur (none) -> Wurth; MFR 865060445005 -> 865 060 445 005
- C203, C204: Fournisseur (none) -> Wurth; MFR 865060442002 -> 865 060 442 002
- C205: footprint Capacitor_SMD:C_0402_1005Metric_Pad0.74x0.62mm_HandSolder -> Capacitor_SMD:C_0402_1005Metric; Fournisseur (none) -> Wurth; MFR (none) -> 885 012 205 050
- C207: renamed from C206; footprint Capacitor_SMD:C_0402_1005Metric_Pad0.74x0.62mm_HandSolder -> Capacitor_SMD:C_0402_1005Metric; Fournisseur (none) -> Wurth; MFR (none) -> 885 012 105 018
- C208: renamed from C207; footprint Capacitor_SMD:C_0402_1005Metric_Pad0.74x0.62mm_HandSolder -> Capacitor_SMD:C_0402_1005Metric; Fournisseur (none) -> Wurth; MFR (none) -> 885 012 105 018
- C209: renamed from C208; footprint Capacitor_SMD:C_0402_1005Metric_Pad0.74x0.62mm_HandSolder -> Capacitor_SMD:C_0402_1005Metric; Fournisseur (none) -> Wurth; MFR (none) -> 885 012 205 048
- C210: renamed from C209; footprint Capacitor_SMD:C_0402_1005Metric_Pad0.74x0.62mm_HandSolder -> Capacitor_SMD:C_0402_1005Metric; Fournisseur (none) -> Wurth; MFR (none) -> 885 012 205 048
- C211: renamed from C210; footprint Capacitor_SMD:C_0402_1005Metric_Pad0.74x0.62mm_HandSolder -> Capacitor_SMD:C_0402_1005Metric; Fournisseur (none) -> Wurth; MFR (none) -> 885 012 205 048
- Q201: Fournisseur (none) -> RS; MFR (none) -> HCPL-315J-500E; Ref (none) -> 174-4163
- Q202, Q203: Fournisseur (none) -> RS; MFR (none) -> IRF540NPBF; Ref (none) -> 914-8154
- R201, R202: footprint Resistor_SMD:R_0402_1005Metric_Pad0.72x0.64mm_HandSolder -> Resistor_SMD:R_0402_1005Metric; Fournisseur (none) -> Stock
- R206: renamed from R203; footprint Resistor_SMD:R_1206_3216Metric_Pad1.30x1.75mm_HandSolder -> Resistor_SMD:R_1206_3216Metric; Fournisseur (none) -> Stock
- R208: renamed from R204; footprint Resistor_SMD:R_1206_3216Metric_Pad1.30x1.75mm_HandSolder -> Resistor_SMD:R_1206_3216Metric; Fournisseur (none) -> Stock
- R210: renamed from R205; footprint Resistor_SMD:R_0402_1005Metric_Pad0.72x0.64mm_HandSolder -> Resistor_SMD:R_0402_1005Metric; Fournisseur (none) -> Stock
- R211: renamed from R206; footprint Resistor_SMD:R_0402_1005Metric_Pad0.72x0.64mm_HandSolder -> Resistor_SMD:R_0402_1005Metric; Fournisseur (none) -> Farnell; MFR (none) -> MCWR04X1001FTL; Ref (none) -> 2446437
- U201, U202: Fournisseur (none) -> Farnell*; MFR (none) -> MPRB2415S/PQQ6W-Q24-D15-S; Ref (none) -> 3652723/4138610
- U204: Fournisseur (none) -> Farnell; MFR (none) -> GO 10-SME/SP3; Ref (none) -> 3796461
- U303: Fournisseur (none) -> RS; MFR (none) -> HCPL-7800A-500E; Ref (none) -> 174-4179
Connections:
- net ARM_OUT: now also R207.2
- net Cmd_H: now also R207.1
- net Cmd_L: now also R209.1
- net GND: now also R209.2
- net ISO_GND: now also R807.2, R807.2, R807.2
- net In_H: now also D804.2 (A)
- net In_L: now also D804.2 (A)
- net PwrEn: now also D804.2 (A)
- new net: D804.1 (K), R807.1 (x3)

Commit message: update pcb
Parts:
- R210: value 160k -> 470k
- renumbered C1 to C?, D804 to D?, R807 to R?
Other:
- note added: "HCPL-7800A Gain : 8V/V (differential) 4V/V (signe ended) Offset : 2.5V"
- note removed: "HCPL-7800A Gain : 8V/V"
- moved on the sheet: C205, R210, R211, U303
