File: Inverter_KiCAD/V_Power_LED.kicad_sch (KiCad schematic)
At the start: 6 parts

Commit message: update pcb
Parts:
- renumbered D804 to D?, R807 to R?
Changed lines of the file:
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@@
   (symbol (lib_id "Device:R_Small") (at 165.1 105.41 90) (unit 1)
     (in_bom yes) (on_board yes) (dnp no)
-    (property "Reference" "R807" (at 165.1 107.95 90)
+    (property "Reference" "R?" (at 165.1 107.95 90)
       (effects (font (size 1.27 1.27)))
     )
@@
       (project "Inverter_KiCAD"
         (path "/5e6c1e3f-0815-454a-8acb-8e3e2d064875/98f7f190-4cd6-4f5a-9ea2-2a00e81dec72"
-          (reference "R807") (unit 1)
-        )
-        (path "/5e6c1e3f-0815-454a-8acb-8e3e2d064875/9da1d24f-0210-4c44-b691-d03fb3165448"
-          (reference "R205") (unit 1)
-        )
-        (path "/5e6c1e3f-0815-454a-8acb-8e3e2d064875/7e6a23ff-8591-450f-995d-37af863aff63"
-          (reference "R305") (unit 1)
-        )
-        (path "/5e6c1e3f-0815-454a-8acb-8e3e2d064875/9544454d-ec1d-4fae-9228-d7a31bd25ddf"
-          (reference "R405") (unit 1)
-        )
-        (path "/5e6c1e3f-0815-454a-8acb-8e3e2d064875/0406dcca-4785-4175-98fc-8c562936c28c"
-          (reference "R502") (unit 1)
+          (reference "R?") (unit 1)
+        )
+        (path "/5e6c1e3f-0815-454a-8acb-8e3e2d064875/9da1d24f-0210-4c44-b691-d03fb3165448"
+          (reference "R?") (unit 1)
+        )
+        (path "/5e6c1e3f-0815-454a-8acb-8e3e2d064875/7e6a23ff-8591-450f-995d-37af863aff63"
+          (reference "R?") (unit 1)
+        )
+        (path "/5e6c1e3f-0815-454a-8acb-8e3e2d064875/9544454d-ec1d-4fae-9228-d7a31bd25ddf"
+          (reference "R?") (unit 1)
         )
         (path "/5e6c1e3f-0815-454a-8acb-8e3e2d064875/f6f2a29f-f026-4c21-995d-91977554a240"
@@
   (symbol (lib_id "Device:R_Small") (at 165.1 96.52 90) (unit 1)
     (in_bom yes) (on_board yes) (dnp no)
-    (property "Reference" "R807" (at 165.1 99.06 90)
+    (property "Reference" "R?" (at 165.1 99.06 90)
       (effects (font (size 1.27 1.27)))
     )
@@
       (project "Inverter_KiCAD"
         (path "/5e6c1e3f-0815-454a-8acb-8e3e2d064875/98f7f190-4cd6-4f5a-9ea2-2a00e81dec72"
-          (reference "R807") (unit 1)
-        )
-        (path "/5e6c1e3f-0815-454a-8acb-8e3e2d064875/9da1d24f-0210-4c44-b691-d03fb3165448"
-          (reference "R205") (unit 1)
-        )
-        (path "/5e6c1e3f-0815-454a-8acb-8e3e2d064875/7e6a23ff-8591-450f-995d-37af863aff63"
-          (reference "R305") (unit 1)
-        )
-        (path "/5e6c1e3f-0815-454a-8acb-8e3e2d064875/9544454d-ec1d-4fae-9228-d7a31bd25ddf"
-          (reference "R405") (unit 1)
-        )
-        (path "/5e6c1e3f-0815-454a-8acb-8e3e2d064875/0406dcca-4785-4175-98fc-8c562936c28c"
-          (reference "R501") (unit 1)
+          (reference "R?") (unit 1)
+        )
+        (path "/5e6c1e3f-0815-454a-8acb-8e3e2d064875/9da1d24f-0210-4c44-b691-d03fb3165448"
+          (reference "R?") (unit 1)
+        )
+        (path "/5e6c1e3f-0815-454a-8acb-8e3e2d064875/7e6a23ff-8591-450f-995d-37af863aff63"
+          (reference "R?") (unit 1)
+        )
+        (path "/5e6c1e3f-0815-454a-8acb-8e3e2d064875/9544454d-ec1d-4fae-9228-d7a31bd25ddf"
+          (reference "R?") (unit 1)
         )
         (path "/5e6c1e3f-0815-454a-8acb-8e3e2d064875/f6f2a29f-f026-4c21-995d-91977554a240"
@@
   (symbol (lib_id "Device:LED") (at 156.21 114.3 180) (unit 1)
     (in_bom yes) (on_board yes) (dnp no)
-    (property "Reference" "D804" (at 156.21 116.84 0)
+    (property "Reference" "D?" (at 156.21 116.84 0)
       (effects (font (size 1.27 1.27)))
     )
@@
       (project "Inverter_KiCAD"
         (path "/5e6c1e3f-0815-454a-8acb-8e3e2d064875/98f7f190-4cd6-4f5a-9ea2-2a00e81dec72"
-          (reference "D804") (unit 1)
-        )
-        (path "/5e6c1e3f-0815-454a-8acb-8e3e2d064875/9da1d24f-0210-4c44-b691-d03fb3165448"
-          (reference "D203") (unit 1)
-        )
-        (path "/5e6c1e3f-0815-454a-8acb-8e3e2d064875/7e6a23ff-8591-450f-995d-37af863aff63"
-          (reference "D303") (unit 1)
-        )
-        (path "/5e6c1e3f-0815-454a-8acb-8e3e2d064875/9544454d-ec1d-4fae-9228-d7a31bd25ddf"
-          (reference "D403") (unit 1)
-        )
-        (path "/5e6c1e3f-0815-454a-8acb-8e3e2d064875/0406dcca-4785-4175-98fc-8c562936c28c"
-          (reference "D503") (unit 1)
+          (reference "D?") (unit 1)
+        )
+        (path "/5e6c1e3f-0815-454a-8acb-8e3e2d064875/9da1d24f-0210-4c44-b691-d03fb3165448"
+          (reference "D?") (unit 1)
+        )
+        (path "/5e6c1e3f-0815-454a-8acb-8e3e2d064875/7e6a23ff-8591-450f-995d-37af863aff63"
+          (reference "D?") (unit 1)
+        )
+        (path "/5e6c1e3f-0815-454a-8acb-8e3e2d064875/9544454d-ec1d-4fae-9228-d7a31bd25ddf"
+          (reference "D?") (unit 1)
         )
         (path "/5e6c1e3f-0815-454a-8acb-8e3e2d064875/f6f2a29f-f026-4c21-995d-91977554a240"
@@
   (symbol (lib_id "Device:LED") (at 156.21 105.41 180) (unit 1)
     (in_bom yes) (on_board yes) (dnp no)
-    (property "Reference" "D804" (at 156.21 107.95 0)
+    (property "Reference" "D?" (at 156.21 107.95 0)
       (effects (font (size 1.27 1.27)))
     )
@@
       (project "Inverter_KiCAD"
         (path "/5e6c1e3f-0815-454a-8acb-8e3e2d064875/98f7f190-4cd6-4f5a-9ea2-2a00e81dec72"
-          (reference "D804") (unit 1)
-        )
-        (path "/5e6c1e3f-0815-454a-8acb-8e3e2d064875/9da1d24f-0210-4c44-b691-d03fb3165448"
-          (reference "D203") (unit 1)
-        )
-        (path "/5e6c1e3f-0815-454a-8acb-8e3e2d064875/7e6a23ff-8591-450f-995d-37af863aff63"
-          (reference "D303") (unit 1)
-        )
-        (path "/5e6c1e3f-0815-454a-8acb-8e3e2d064875/9544454d-ec1d-4fae-9228-d7a31bd25ddf"
-          (reference "D403") (unit 1)
-        )
-        (path "/5e6c1e3f-0815-454a-8acb-8e3e2d064875/0406dcca-4785-4175-98fc-8c562936c28c"
-          (reference "D502") (unit 1)
+          (reference "D?") (unit 1)
+        )
+        (path "/5e6c1e3f-0815-454a-8acb-8e3e2d064875/9da1d24f-0210-4c44-b691-d03fb3165448"
+          (reference "D?") (unit 1)
+        )
+        (path "/5e6c1e3f-0815-454a-8acb-8e3e2d064875/7e6a23ff-8591-450f-995d-37af863aff63"
+          (reference "D?") (unit 1)
+        )
+        (path "/5e6c1e3f-0815-454a-8acb-8e3e2d064875/9544454d-ec1d-4fae-9228-d7a31bd25ddf"
+          (reference "D?") (unit 1)
         )
         (path "/5e6c1e3f-0815-454a-8acb-8e3e2d064875/f6f2a29f-f026-4c21-995d-91977554a240"
@@
   (symbol (lib_id "Device:LED") (at 156.21 96.52 180) (unit 1)
     (in_bom yes) (on_board yes) (dnp no)
-    (property "Reference" "D804" (at 156.21 99.06 0)
+    (property "Reference" "D?" (at 156.21 99.06 0)
       (effects (font (size 1.27 1.27)))
     )
@@
       (project "Inverter_KiCAD"
         (path "/5e6c1e3f-0815-454a-8acb-8e3e2d064875/98f7f190-4cd6-4f5a-9ea2-2a00e81dec72"
-          (reference "D804") (unit 1)
-        )
-        (path "/5e6c1e3f-0815-454a-8acb-8e3e2d064875/9da1d24f-0210-4c44-b691-d03fb3165448"
-          (reference "D203") (unit 1)
-        )
-        (path "/5e6c1e3f-0815-454a-8acb-8e3e2d064875/7e6a23ff-8591-450f-995d-37af863aff63"
-          (reference "D303") (unit 1)
-        )
-        (path "/5e6c1e3f-0815-454a-8acb-8e3e2d064875/9544454d-ec1d-4fae-9228-d7a31bd25ddf"
-          (reference "D403") (unit 1)
-        )
-        (path "/5e6c1e3f-0815-454a-8acb-8e3e2d064875/0406dcca-4785-4175-98fc-8c562936c28c"
-          (reference "D501") (unit 1)
+          (reference "D?") (unit 1)
+        )
+        (path "/5e6c1e3f-0815-454a-8acb-8e3e2d064875/9da1d24f-0210-4c44-b691-d03fb3165448"
+          (reference "D?") (unit 1)
+        )
+        (path "/5e6c1e3f-0815-454a-8acb-8e3e2d064875/7e6a23ff-8591-450f-995d-37af863aff63"
+          (reference "D?") (unit 1)
+        )
+        (path "/5e6c1e3f-0815-454a-8acb-8e3e2d064875/9544454d-ec1d-4fae-9228-d7a31bd25ddf"
+          (reference "D?") (unit 1)
         )
         (path "/5e6c1e3f-0815-454a-8acb-8e3e2d064875/f6f2a29f-f026-4c21-995d-91977554a240"
@@
   (symbol (lib_id "Device:R_Small") (at 165.1 114.3 90) (unit 1)
     (in_bom yes) (on_board yes) (dnp no)
-    (property "Reference" "R807" (at 165.1 116.84 90)
+    (property "Reference" "R?" (at 165.1 116.84 90)
       (effects (font (size 1.27 1.27)))
     )
@@
       (project "Inverter_KiCAD"
         (path "/5e6c1e3f-0815-454a-8acb-8e3e2d064875/98f7f190-4cd6-4f5a-9ea2-2a00e81dec72"
-          (reference "R807") (unit 1)
-        )
-        (path "/5e6c1e3f-0815-454a-8acb-8e3e2d064875/9da1d24f-0210-4c44-b691-d03fb3165448"
-          (reference "R205") (unit 1)
-        )
-        (path "/5e6c1e3f-0815-454a-8acb-8e3e2d064875/7e6a23ff-8591-450f-995d-37af863aff63"
-          (reference "R305") (unit 1)
-        )
-        (path "/5e6c1e3f-0815-454a-8acb-8e3e2d064875/9544454d-ec1d-4fae-9228-d7a31bd25ddf"
-          (reference "R405") (unit 1)
-        )
-        (path "/5e6c1e3f-0815-454a-8acb-8e3e2d064875/0406dcca-4785-4175-98fc-8c562936c28c"
-          (reference "R503") (unit 1)
-        )
-        (path "/5e6c1e3f-0815-454a-8acb-8e3e2d064875/f6f2a29f-f026-4c21-995d-91977554a240"
+          (reference "R?") (unit 1)
+        )
+        (path "/5e6c1e3f-0815-454a-8acb-8e3e2d064875/9da1d24f-0210-4c44-b691-d03fb3165448"
+          (reference "R?") (unit 1)
+        )
+        (path "/5e6c1e3f-0815-454a-8acb-8e3e2d064875/7e6a23ff-8591-450f-995d-37af863aff63"
+          (reference "R?") (unit 1)
+        )
+        (path "/5e6c1e3f-0815-454a-8acb-8e3e2d064875/9544454d-ec1d-4fae-9228-d7a31bd25ddf"
+          (reference "R?") (unit 1)
+        )
+        (path "/5e6c1e3f-0815-454a-8acb-8e3e2d064875/f6f2a29f-f026-4c21-995d-91977554a240"
