File: Inverter_KiCAD/encoderMotor.kicad_sch (KiCad schematic)
At the start: 4 parts, among them J3 DE9_Receptacle_MountingHoles, J4 Conn_01x03, U1 MAX3097ECSE+

Commit message: update pcb
Parts:
- removed J4: Conn_01x03, Connector_PinHeader_2.54mm:PinHeader_1x03_P2.54mm_Vertical, symbol Connector_Generic:Conn_01x03
- C1301: renamed from C4; footprint Capacitor_SMD:C_0402_1005Metric_Pad0.74x0.62mm_HandSolder -> Capacitor_SMD:C_0402_1005Metric; Fournisseur (none) -> Wurth; MFR (none) -> 885 012 105 018
- J1301: renamed from J3; Fournisseur (none) -> Wurth; MFR 618009231421 -> 618 009 231 421
- U1301: renamed from U1; Fournisseur (none) -> Farnell; MFR (none) -> MAX3097ECSE+; Ref (none) -> 2518786
Connections:
- net A: now also J1301.5; no longer J1301.1
- net B: now also J1301.9; no longer J1301.6
- net ISO_3V3: now also J1301.1
- net ISO_GND: now also J1301.2; no longer J1301.4
- net VCC_Enc: no longer J1301.5
- net Z: now also J1301.7; no longer J1301.8
- net /A: now also J1301.4; no longer J1301.2
- net /B: now also J1301.8; no longer J1301.7
- net /Z: now also J1301.6; no longer J1301.9
Other:
- moved on the sheet: J1301
