File: Inverter_KiCAD/pwrSupply.kicad_sch (KiCad schematic)
At the start: 7 parts, among them J501 PX0580-PC-12132, U501 MP-LD30-23B12R2, U502 173010542, U503 AZ1117-3.3

Commit message: end of sch, start pcb
Parts:
- F501: footprint (none) -> Custom:0031.8201
- U502: footprint (none) -> Custom:173010578
Other:
- company: (none) -> ENSEA
- title: (none) -> AAP Inverter
Changed lines of the file:
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@@
 (kicad_sch (version 20230121) (generator eeschema)
   (paper "A4")
+  (title_block
+    (title "AAP Inverter")
+    (date "2023-05-01")
+    (company "ENSEA")
+  )
   (junction (at 231.14 34.29) (diameter 0) (color 0 0 0 0)
   )
@@
   )
   (symbol (lib_id "Device:Fuse") (at 45.72 43.18 90) (unit 1)
-    (in_bom yes) (on_board yes) (dnp no) (fields_autoplaced)
+    (in_bom yes) (on_board yes) (dnp no)
     (property "Reference" "F501" (at 45.72 38.1 90)
       (effects (font (size 1.27 1.27)))
@@
       (effects (font (size 1.27 1.27)))
     )
-    (property "Footprint" "" (at 45.72 44.958 90)
+    (property "Footprint" "Custom:0031.8201" (at 45.72 52.07 90)
       (effects (font (size 1.27 1.27)) hide)
     )
@@
       (effects (font (size 1.524 1.524)))
     )
-    (property "Footprint" "" (at 149.86 49.53 0)
-      (effects (font (size 1.27 1.27) italic) hide)
-    )
+    (property "Footprint" "Custom:173010578" (at 149.86 49.53 0)
+      (effects (font (size 1.27 1.27) italic) hide)
+    )

Commit message: apply changes
Connections:
- net Earth: no longer names the net of J501.2 (Earth)
- no-connect marks 0 -> 1
Changed lines of the file:
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@@
   (junction (at 205.74 34.29) (diameter 0) (color 0 0 0 0)
   )
+  (no_connect (at 34.29 40.64))
   (wire (pts (xy 123.19 36.83) (xy 125.73 36.83))
     (stroke (width 0) (type default))
@@
   )
   (wire (pts (xy 219.71 45.72) (xy 219.71 41.91))
-    (stroke (width 0) (type default))
-  )
-  (wire (pts (xy 34.29 40.64) (xy 35.56 40.64))
     (stroke (width 0) (type default))
   )
@@
     (effects (font (size 1.27 1.27)) (justify right))
   )
-  (symbol (lib_id "power:Earth") (at 35.56 40.64 90) (unit 1)
-    (in_bom yes) (on_board yes) (dnp no) (fields_autoplaced)
-    (property "Reference" "#PWR0501" (at 41.91 40.64 0)
-      (effects (font (size 1.27 1.27)) hide)
-    )
-    (property "Value" "Earth" (at 39.37 40.64 0)
-      (effects (font (size 1.27 1.27)) hide)
-    )
-    (property "Footprint" "" (at 35.56 40.64 0)
-      (effects (font (size 1.27 1.27)) hide)
-    )
-    (property "Datasheet" "~" (at 35.56 40.64 0)
-      (effects (font (size 1.27 1.27)) hide)
-    )
-    (pin "1")
-    (instances
-      (project "Inverter_KiCAD"
-        (path "/5e6c1e3f-0815-454a-8acb-8e3e2d064875/0406dcca-4785-4175-98fc-8c562936c28c"
-          (reference "#PWR0501") (unit 1)
-        )
-      )
-    )
-  )
   (symbol (lib_id "Device:C_Polarized") (at 231.14 40.64 0) (unit 1)

Commit message: update pcb
Parts:
- added D804 (x3): Red LED, LED_SMD:LED_0603_1608Metric, symbol Device:LED
- added R807: 2k7, Resistor_SMD:R_0402_1005Metric, symbol Device:R_Small
- added R807: 390, Resistor_SMD:R_0402_1005Metric, symbol Device:R_Small
- added R807: 680, Resistor_SMD:R_0402_1005Metric, symbol Device:R_Small
- C501: Fournisseur (none) -> Wurth; MFR 865060440001 -> 865 060 440 001
- C502: Fournisseur (none) -> Wurth; MFR 865060442002 -> 865 060 442 002
- F501: Fournisseur (none) -> Wurth; MFR (none) -> 696 108 003 002
- J501: Fournisseur (none) -> RS; MFR (none) -> PX0580/PC/12132; Ref (none) -> 261-5840
- U501: Fournisseur (none) -> Farnell; MFR (none) -> MP-LD30-23B15R2; Ref (none) -> 3780527
- U502: Fournisseur (none) -> Wurth; MFR (none) -> 173 010 542
- U503: Fournisseur (none) -> RS; MFR (none) -> AZ1117H-3.3TRE1; Ref (none) -> 921-0701
Connections:
- net ISO_15V: now also D804.2 (A)
- net ISO_3V3: now also D804.2 (A)
- net ISO_5V: now also D804.2 (A)
- net ISO_GND: now also R807.2, R807.2, R807.2
- new net: D804.1 (K), R807.1 (x3)

Commit message: update pcb
Parts:
- renumbered D804 to D?, R807 to R?
Other:
- moved on the sheet: D?, R?
